File: PCBs/BindingPosts/v1.0.0/BindingPosts.kicad_pcb (KiCad board)
At the start: 2 copper layers, 100 x 60 mm, 25 parts, among them J1 Conn_01x02_Male, J2 Conn_01x02_Male, J3 Conn_01x02_Male, J4 Conn_01x02_Male, J5 Conn_01x02_Male

Commit message: Adding images
Other:
- board text added: "BINDING POSTS VER 1.0.0"
- board text removed: "BINDING POSTS VER 1.0.6"
Changed lines of the file:
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@@
     (effects (font (size 0.7 0.7) (thickness 0.1)) (justify right))
   )
-  (gr_text "BINDING POSTS VER 1.0.6" (at 138 42) (layer "F.SilkS")
+  (gr_text "BINDING POSTS VER 1.0.0" (at 138 42) (layer "F.SilkS")
     (effects (font (size 0.7 0.7) (thickness 0.1)) (justify right))
   )
