File: PCBs/SOIC DIP/SOIC DIP.kicad_pcb (KiCad board)
At the start: 2 copper layers, 15 x 15 mm, 4 parts, among them U1 OPA2134, U2 OPA2134

Commit message: Removing gerbers and backups
Other:
- board size 15 x 15 mm -> 13 x 14.5 mm
