File: PCBs/Channel Amplifier/1.0/PowerAmp.kicad_sch (KiCad schematic)
At the start: 42 parts, among them J1 Conn_01x02_Male, J2 Conn_01x02_Male, J3 Conn_01x02_Male, J4 Conn_01x02_Male, J5 Conn_01x03_Male, J6 Conn_01x02_Male, J7 Conn_01x02_Male, J8 Conn_01x03_Male, J9 Conn_01x02_Male, U1 TMP100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

Commit message: Updates
Parts:
- C2: value 10N -> 100N
Changed lines of the file:
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@@
       (effects (font (size 1.27 1.27)) (justify right))
     )
-    (property "Value" "10N" (id 1) (at 251.333 31.1085 0)
+    (property "Value" "100N" (id 1) (at 251.333 31.1085 0)
       (effects (font (size 1.27 1.27)) (justify right))
     )
@@
     )
     (path "/93c239a2-b113-4b85-8561-44058676d21b"
-      (reference "C2") (unit 1) (value "10N") (footprint "Resistor_SMD:R_0805_2012Metric_Pad1.20x1.40mm_HandSolder")
+      (reference "C2") (unit 1) (value "100N") (footprint "Resistor_SMD:R_0805_2012Metric_Pad1.20x1.40mm_HandSolder")
     )
     (path "/fdc886c0-31da-4fe9-add1-d3334adcebd6"
