File: PCBs/Channel Amplifier/1.0/PowerAmp.kicad_pcb (KiCad board)
At the start: 2 copper layers, 55 x 55 mm, 42 parts, among them J1 Conn_01x02_Male, J2 Conn_01x02_Male, J3 Conn_01x02_Male, J4 Conn_01x02_Male, J5 Conn_01x03_Male, J6 Conn_01x02_Male, J7 Conn_01x02_Male, J8 Conn_01x03_Male, J9 Conn_01x02_Male, U1 TMP100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

Commit message: KiCAD 7 updates
Parts:
- C2: value 10N -> 100N
Routing:
- net PGND: track 28.5 -> 26.8 mm

Commit message: Major updates
Parts:
- added U3: LM4766, Package_TO_SOT_THT:TO-220-15_P2.54x2.54mm_StaggerOdd_Lead4.58mm_Vertical, F.Cu at (1.49, 9.86)
Changed lines of the file:
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@@
   (net 25 "CH1GND")
   (net 26 "OPAMP_NEG")
+  (net 27 "unconnected-(U3-Pad1)")
+  (net 28 "unconnected-(U3A-V+-Pad2)")
+  (net 29 "unconnected-(U3-Pad3)")
+  (net 30 "unconnected-(U3A-V--Pad4)")
+  (net 31 "unconnected-(U3A-GND-Pad5)")
+  (net 32 "unconnected-(U3A-MUTE-Pad6)")
+  (net 33 "unconnected-(U3A---Pad7)")
+  (net 34 "unconnected-(U3A-+-Pad8)")
+  (net 35 "unconnected-(U3A-NC-Pad9)")
+  (net 36 "unconnected-(U3B-GND-Pad10)")
+  (net 37 "unconnected-(U3B-MUTE-Pad11)")
+  (net 38 "unconnected-(U3B---Pad12)")
+  (net 39 "unconnected-(U3B-+-Pad13)")
+  (net 40 "unconnected-(U3B-NC-Pad14)")
+  (net 41 "unconnected-(U3B-V+-Pad15)")
   (footprint "Resistor_THT:R_Axial_DIN0207_L6.3mm_D2.5mm_P10.16mm_Horizontal" (layer "F.Cu")
     (at 94.5 98.37 -90)
@@
       (offset (xyz 0 0 0))
       (scale (xyz 1 1 1))
+      (rotate (xyz 0 0 0))
+    )
+  )
+  (footprint "Package_TO_SOT_THT:TO-220-15_P2.54x2.54mm_StaggerOdd_Lead4.58mm_Vertical" (layer "F.Cu")
+    (at 1.485 9.855)
+    (descr "TO-220-15, Vertical, RM 1.27mm, staggered type-1, see http://www.st.com/resource/en/datasheet/l298.pdf")
+    (tags "TO-220-15 Vertical RM 1.27mm staggered type-1")
+    (property "Sheetfile" "PowerAmp.kicad_sch")
+    (property "Sheetname" "")
+    (property "ki_description" "Overture Audio Power Amplifier Series Dual 40W Audio Power Amplifier with Mute, TO-220-15")
+    (property "ki_keywords" "audio amplifier 2ch")
+    (attr through_hole)
+    (fp_text reference "U3" (at 8.89 -10.7) (layer "F.SilkS")
+        (effects (font (size 1 1) (thickness 0.15)))
+    )
+    (fp_text value "LM4766" (at 8.89 2.15) (layer "F.Fab")
+        (effects (font (size 1 1) (thickness 0.15)))
+    )
+    (fp_text user "${REFERENCE}" (at 8.89 -10.7) (layer "F.Fab")
+        (effects (font (size 1 1) (thickness 0.15)))
+    )
+    (fp_line (start -1.33 -9.7) (end -1.33 -4.459)
+      (stroke (width 0.12) (type solid)) (layer "F.SilkS"))
+    (fp_line (start -1.33 -9.7) (end 19.11 -9.7)
+      (stroke (width 0.12) (type solid)) (layer "F.SilkS"))
+    (fp_line (start -1.33 -7.86) (end 19.11 -7.86)
+      (stroke (width 0.12) (type solid)) (layer "F.SilkS"))
+    (fp_line (start -1.33 -4.459) (end 0.346 -4.459)
+      (stroke (width 0.12) (type solid)) (layer "F.SilkS"))
+    (fp_line (start 0 -4.459) (end 0 -1.05)
+      (stroke (width 0.12) (type solid)) (layer "F.SilkS"))
+    (fp_line (start 2.195 -4.459) (end 2.886 -4.459)
+      (stroke (width 0.12) (type solid)) (layer "F.SilkS"))
+    (fp_line (start 2.54 -4.459) (end 2.54 -1.065)
+      (stroke (width 0.12) (type solid)) (layer "F.SilkS"))
+    (fp_line (start 4.735 -4.459) (end 5.426 -4.459)
+      (stroke (width 0.12) (type solid)) (layer "F.SilkS"))
+    (fp_line (start 5.08 -4.459) (end 5.08 -1.065)
+      (stroke (width 0.12) (type solid)) (layer "F.SilkS"))
+    (fp_line (start 7.041 -9.7) (end 7.041 -7.86)
+      (stroke (width 0.12) (type solid)) (layer "F.SilkS"))
+    (fp_line (start 7.275 -4.459) (end 7.966 -4.459)
+      (stroke (width 0.12) (type solid)) (layer "F.SilkS"))
+    (fp_line (start 7.62 -4.459) (end 7.62 -1.065)
+      (stroke (width 0.12) (type solid)) (layer "F.SilkS"))
+    (fp_line (start 9.815 -4.459) (end 10.506 -4.459)
+      (stroke (width 0.12) (type solid)) (layer "F.SilkS"))
+    (fp_line (start 10.16 -4.459) (end 10.16 -1.065)
+      (stroke (width 0.12) (type solid)) (layer "F.SilkS"))
+    (fp_line (start 10.74 -9.7) (end 10.74 -7.86)
+      (stroke (width 0.12) (type solid)) (layer "F.SilkS"))
+    (fp_line (start 12.355 -4.459) (end 13.046 -4.459)
+      (stroke (width 0.12) (type solid)) (layer "F.SilkS"))
+    (fp_line (start 12.7 -4.459) (end 12.7 -1.065)
+      (stroke (width 0.12) (type solid)) (layer "F.SilkS"))
+    (fp_line (start 14.895 -4.459) (end 15.586 -4.459)
+      (stroke (width 0.12) (type solid)) (layer "F.SilkS"))
+    (fp_line (start 15.24 -4.459) (end 15.24 -1.065)
+      (stroke (width 0.12) (type solid)) (layer "F.SilkS"))
+    (fp_line (start 17.435 -4.459) (end 19.11 -4.459)
+      (stroke (width 0.12) (type solid)) (layer "F.SilkS"))
+    (fp_line (start 17.78 -4.459) (end 17.78 -1.065)
+      (stroke (width 0.12) (type solid)) (layer "F.SilkS"))
+    (fp_line (start 19.11 -9.7) (end 19.11 -4.459)
+      (stroke (width 0.12) (type solid)) (layer "F.SilkS"))
+    (fp_line (start -1.46 -9.83) (end -1.46 1.16)
+      (stroke (width 0.05) (type solid)) (layer "F.CrtYd"))
+    (fp_line (start -1.46 1.16) (end 19.25 1.16)
+      (stroke (width 0.05) (type solid)) (layer "F.CrtYd"))
+    (fp_line (start 19.25 -9.83) (end -1.46 -9.83)
+      (stroke (width 0.05) (type solid)) (layer "F.CrtYd"))
+    (fp_line (start 19.25 1.16) (end 19.25 -9.83)
+      (stroke (width 0.05) (type solid)) (layer "F.CrtYd"))
+    (fp_line (start -1.21 -9.58) (end -1.21 -4.58)
+      (stroke (width 0.1) (type solid)) (layer "F.Fab"))
+    (fp_line (start -1.21 -7.98) (end 18.99 -7.98)
+      (stroke (width 0.1) (type solid)) (layer "F.Fab"))
+    (fp_line (start -1.21 -4.58) (end 18.99 -4.58)
+      (stroke (width 0.1) (type solid)) (layer "F.Fab"))
+    (fp_line (start 0 -4.58) (end 0 0)
+      (stroke (width 0.1) (type solid)) (layer "F.Fab"))
+    (fp_line (start 2.54 -4.58) (end 2.54 0)
+      (stroke (width 0.1) (type solid)) (layer "F.Fab"))
+    (fp_line (start 5.08 -4.58) (end 5.08 0)
+      (stroke (width 0.1) (type solid)) (layer "F.Fab"))
+    (fp_line (start 7.04 -9.58) (end 7.04 -7.98)
+      (stroke (width 0.1) (type solid)) (layer "F.Fab"))
+    (fp_line (start 7.62 -4.58) (end 7.62 0)
+      (stroke (width 0.1) (type solid)) (layer "F.Fab"))
+    (fp_line (start 10.16 -4.58) (end 10.16 0)
+      (stroke (width 0.1) (type solid)) (layer "F.Fab"))
+    (fp_line (start 10.74 -9.58) (end 10.74 -7.98)
+      (stroke (width 0.1) (type solid)) (layer "F.Fab"))
+    (fp_line (start 12.7 -4.58) (end 12.7 0)
+      (stroke (width 0.1) (type solid)) (layer "F.Fab"))
+    (fp_line (start 15.24 -4.58) (end 15.24 0)
+      (stroke (width 0.1) (type solid)) (layer "F.Fab"))
+    (fp_line (start 17.78 -4.58) (end 17.78 0)
+      (stroke (width 0.1) (type solid)) (layer "F.Fab"))
+    (fp_line (start 18.99 -9.58) (end -1.21 -9.58)
+      (stroke (width 0.1) (type solid)) (layer "F.Fab"))
+    (fp_line (start 18.99 -4.58) (end 18.99 -9.58)
+      (stroke (width 0.1) (type solid)) (layer "F.Fab"))
+    (pad "1" thru_hole rect (at 0 0) (size 1.8 1.8) (drill 1) (layers "*.Cu" "*.Mask")
+      (net 27 "unconnected-(U3-Pad1)") (pintype "output"))
+    (pad "2" thru_hole oval (at 1.27 -5.08) (size 1.8 1.8) (drill 1) (layers "*.Cu" "*.Mask")
+      (net 28 "unconnected-(U3A-V+-Pad2)") (pinfunction "V+") (pintype "power_in"))
+    (pad "3" thru_hole oval (at 2.54 0) (size 1.8 1.8) (drill 1) (layers "*.Cu" "*.Mask")
+      (net 29 "unconnected-(U3-Pad3)") (pintype "output"))
+    (pad "4" thru_hole oval (at 3.81 -5.08) (size 1.8 1.8) (drill 1) (layers "*.Cu" "*.Mask")
+      (net 30 "unconnected-(U3A-V--Pad4)") (pinfunction "V-") (pintype "power_in"))
+    (pad "5" thru_hole oval (at 5.08 0) (size 1.8 1.8) (drill 1) (layers "*.Cu" "*.Mask")
+      (net 31 "unconnected-(U3A-GND-Pad5)") (pinfunction "GND") (pintype "power_in"))
+    (pad "6" thru_hole oval (at 6.35 -5.08) (size 1.8 1.8) (drill 1) (layers "*.Cu" "*.Mask")
+      (net 32 "unconnected-(U3A-MUTE-Pad6)") (pinfunction "MUTE") (pintype "input"))
+    (pad "7" thru_hole oval (at 7.62 0) (size 1.8 1.8) (drill 1) (layers "*.Cu" "*.Mask")
+      (net 33 "unconnected-(U3A---Pad7)") (pinfunction "-") (pintype "input"))
+    (pad "8" thru_hole oval (at 8.89 -5.08) (size 1.8 1.8) (drill 1) (layers "*.Cu" "*.Mask")
+      (net 34 "unconnected-(U3A-+-Pad8)") (pinfunction "+") (pintype "input"))
+    (pad "9" thru_hole oval (at 10.16 0) (size 1.8 1.8) (drill 1) (layers "*.Cu" "*.Mask")
+      (net 35 "unconnected-(U3A-NC-Pad9)") (pinfunction "NC") (pintype "no_connect"))
+    (pad "10" thru_hole oval (at 11.43 -5.08) (size 1.8 1.8) (drill 1) (layers "*.Cu" "*.Mask")
+      (net 36 "unconnected-(U3B-GND-Pad10)") (pinfunction "GND") (pintype "power_in"))
+    (pad "11" thru_hole oval (at 12.7 0) (size 1.8 1.8) (drill 1) (layers "*.Cu" "*.Mask")
+      (net 37 "unconnected-(U3B-MUTE-Pad11)") (pinfunction "MUTE") (pintype "input"))
+    (pad "12" thru_hole oval (at 13.97 -5.08) (size 1.8 1.8) (drill 1) (layers "*.Cu" "*.Mask")
+      (net 38 "unconnected-(U3B---Pad12)") (pinfunction "-") (pintype "input"))
+    (pad "13" thru_hole oval (at 15.24 0) (size 1.8 1.8) (drill 1) (layers "*.Cu" "*.Mask")
+      (net 39 "unconnected-(U3B-+-Pad13)") (pinfunction "+") (pintype "input"))
+    (pad "14" thru_hole oval (at 16.51 -5.08) (size 1.8 1.8) (drill 1) (layers "*.Cu" "*.Mask")
+      (net 40 "unconnected-(U3B-NC-Pad14)") (pinfunction "NC") (pintype "no_connect"))
+    (pad "15" thru_hole oval (at 17.78 0) (size 1.8 1.8) (drill 1) (layers "*.Cu" "*.Mask")
+      (net 41 "unconnected-(U3B-V+-Pad15)") (pinfunction "V+") (pintype "power_in"))
+    (model "${KICAD6_3DMODEL_DIR}/Package_TO_SOT_THT.3dshapes/TO-220-15_P2.54x2.54mm_StaggerOdd_Lead4.58mm_Vertical.wrl"
+      (offset (xyz 0 0 0))
+      (scale (xyz 1 1 1))
