File: PCBs/DAC/1.0/DAC.kicad_pcb (KiCad board)
At the start: 2 copper layers, 55 x 55 mm, 40 parts, among them J1 Conn_01x02_Male, J10 Conn_01x04_Male, J11 Conn_01x02_Male, J12 Conn_01x02_Male, J13 Conn_01x03_Male, J14 Conn_01x02_Male, J15 Conn_01x02_Male, J2 Conn_01x02_Male, J3 Conn_01x02_Male, J4 Conn_01x02_Male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

Commit message: Updated
Routing:
- net I2S_D4: track 15.6 -> 14.1 mm
