File: PCBs/Microprocessor/1.0/uProcessor.kicad_pcb (KiCad board)
At the start: 2 copper layers, 55 x 95 mm, 109 parts, among them J1 Conn_01x06_Male, J10 Conn_01x02_Male, J11 Conn_01x06_Male, J12 Conn_01x06_Male, J13 Conn_01x02_Male, J14 Conn_01x02_Male, J15 Conn_01x02_Male, J16 Conn_01x02_Male, J17 Conn_01x02_Male, J18 Conn_01x02_Male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

Commit message: Updated
Parts:
- SW1: footprint Button_Switch_SMD:Button_4x4x1.5 -> Components:Button Aliexpress 4x4
- moved SW1 3.73 mm to (119.6, 53.6)
