File: PCBs/BindingPosts/1.0/BindingPosts.kicad_pcb (KiCad board)
At the start: 2 copper layers, 100 x 60 mm, 25 parts, among them J1 Conn_01x02_Male, J2 Conn_01x02_Male, J3 Conn_01x02_Male, J4 Conn_01x02_Male, J5 Conn_01x02_Male

Commit message: Major updates
Other:
- outline, holes or cut-outs redrawn
