File: PCBs/DolbyDecoder/1.1/DolbyDecoder.kicad_pcb (KiCad board)
At the start: 2 copper layers, 55 x 55 mm, 93 parts, among them J1 Conn_01x03_Male, J10 Conn_01x04_Male, J11 Conn_01x03_Male, J12 Conn_01x06_Male, J13 Conn_01x04_Male, J2 Conn_01x03_Male, J3 Conn_01x02, J4 Conn_01x04_Male, J5 Conn_01x02_Male, J6 Conn_01x02_Male, J7 Conn_01x02_Male, J8 Conn_01x02_Male, J9 Conn_01x02_Male, U1 AMS1117-2.5, U2 AMS1117-2.5, U3 SPA130, X1 TXC-7C

Commit message: Updated
Parts:
- added R26: 47R, Resistor_SMD:R_0805_2012Metric_Pad1.20x1.40mm_HandSolder, F.Cu at (166.6, 76.9)
- C17: renamed from C4; value 47U -> 10U
- C18: renamed from C1; value 47U -> 10U
- C22: renamed from C7; value 47U -> 10U
- C33: renamed from C17; value 47U -> 10U
- moved R15 0.60 mm to (161.7, 59.5)
- moved R17 0.60 mm to (161.7, 61.7)
- moved R18 0.60 mm to (161.7, 63.9)
- moved R19 0.60 mm to (161.7, 66.1)
- moved R20 0.60 mm to (161.7, 68.3)
- moved R21 0.60 mm to (161.7, 70.5)
- moved R4 0.10 mm to (128.1, 51.4)
- renumbered C2 to C1, C15 to C10, C29 to C11, C28 to C12, C25 to C13, C24 to C14, C31 to C15, C30 to C16, C23 to C19, C6 to C2, C5 to C21, C19 to C23, C13 to C24, C10 to C25, C22 to C26, C16 to C27, C8 to C28, C12 to C29, C26 to C3, C18 to C30, C11 to C31, C3 to C32, C35 to C34, C34 to C35, C27 to C4, C9 to C5, C21 to C6, C14 to C7, C33 to C8, C32 to C9, D3 to D2, D4 to D3, D2 to D4, H4 to H2, H2 to H4, J9 to J1, J3 to J10, J4 to J11, J7 to J12, J5 to J13, J8 to J2, J12 to J3, J6 to J4, J2 to J5, J13 to J6, J1 to J7, J11 to J8, J10 to J9, R5 to R1, R9 to R10, R8 to R11, R7 to R12, R32 to R13, R22 to R14, R31 to R15, R23 to R16, R30 to R17, R29 to R18, R4 to R2, R26 to R20, R15 to R22, R13 to R23, R17 to R24, R16 to R25, R1 to R27, R25 to R28, R28 to R29, R24 to R30, R20 to R31, R2 to R32, R27 to R34, R18 to R4, R14 to R5, R11 to R6, R6 to R7, R12 to R8, R10 to R9, U3 to U1, U1 to U2, U2 to U3
Connections:
- J6 pad 4: GND -> I2S_D4
- U1 pad 72: unconnected-(U3-PCM_OUT0-Pad72) -> Net-(U1-PCM_OUT0)
Routing:
- net I2S_D4: track 0.00 -> 24.7 mm, vias 0 -> 1
- net Net-(U1-PCM_OUT0): track 0.00 -> 21.3 mm, vias 0 -> 2
- net I2S_D2: track 29.6 -> 28.4 mm
- net Net-(U1-PCMCLK): track 3.07 -> 4.17 mm
- net Net-(U1-LRCLK): track 4.06 -> 4.82 mm
- net GND: track 158.0 -> 158.7 mm
- net Net-(U1-PCM_OUT1): track 3.73 -> 4.33 mm
Other:
- board text added: "DOLBY DECODER VERSION 1.1"
- board text removed: "DOLBY DECODER VERSION 1.0"

Commit message: Major updates
Parts:
- C19: value 10N -> 100N
Routing:
- net Net-(U1-SPDP): track 19.1 -> 19.7 mm
Changed lines of the file:
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@@
         (effects (font (size 0.7 0.7) (thickness 0.1)))
     )
-    (fp_text value "10N" (at 0 1.43 90 unlocked) (layer "F.Fab")
+    (fp_text value "100N" (at 0 1.43 90 unlocked) (layer "F.Fab")
         (effects (font (size 1 1) (thickness 0.15)))
     )
@@
   (segment (start 168.9 56.5) (end 166.9 54.5) (width 0.25) (layer "B.Cu") (net 40))
   (segment (start 168.9 70.4) (end 168.9 56.5) (width 0.25) (layer "B.Cu") (net 40))
-  (segment (start 133.4 49.9) (end 134.2 49.1) (width 0.4) (layer "F.Cu") (net 41))
-  (segment (start 139.3 60.3) (end 140.225 61.225) (width 0.4) (layer "F.Cu") (net 41))
-  (segment (start 141.325 61.225) (end 140.225 61.225) (width 0.4) (layer "F.Cu") (net 41))
   (segment (start 139.3 60.3) (end 139.3 54.4) (width 0.4) (layer "F.Cu") (net 41))
+  (segment (start 137.9 53) (end 135.3 53) (width 0.4) (layer "F.Cu") (net 41))
+  (segment (start 139.3 54.4) (end 137.9 53) (width 0.4) (layer "F.Cu") (net 41))
+  (segment (start 141.325 61.225) (end 140.225 61.225) (width 0.4) (layer "F.Cu") (net 41))
+  (segment (start 133.4 49.9) (end 134.2 49.1) (width 0.4) (layer "F.Cu") (net 41))
   (segment (start 133.4 51.2625) (end 133.4 49.9) (width 0.4) (layer "F.Cu") (net 41))
-  (segment (start 137.8 52.9) (end 136.3 52.9) (width 0.4) (layer "F.Cu") (net 41))
-  (segment (start 139.3 54.4) (end 137.8 52.9) (width 0.4) (layer "F.Cu") (net 41))
+  (segment (start 140.225 61.225) (end 139.3 60.3) (width 0.4) (layer "F.Cu") (net 41))
   (via (at 134.2 49.1) (size 0.8) (drill 0.4) (layers "F.Cu" "B.Cu") (net 41))
-  (via (at 136.3 52.9) (size 0.8) (drill 0.4) (layers "F.Cu" "B.Cu") (net 41))
-  (segment (start 136.3 52.9) (end 134.2 50.8) (width 0.4) (layer "B.Cu") (net 41))
-  (segment (start 134.2 50.8) (end 134.2 49.1) (width 0.4) (layer "B.Cu") (net 41))
+  (via (at 135.3 53) (size 0.8) (drill 0.4) (layers "F.Cu" "B.Cu") (net 41))
+  (segment (start 134.2 49.1) (end 134.2 51.9) (width 0.4) (layer "B.Cu") (net 41))
+  (segment (start 134.2 51.9) (end 135.3 53) (width 0.4) (layer "B.Cu") (net 41))
   (segment (start 140 54.8) (end 140 53.8) (width 0.4) (layer "F.Cu") (net 42))
   (segment (start 141.325 60.575) (end 140.422822 60.575) (width 0.4) (layer "F.Cu") (net 42))
@@
         (xy 126.5 59.2)
         (xy 113.3 59.2)
-        (xy 113.3 48.7)
-        (xy 126.5 48.7)
+        (xy 113.3 47.9)
+        (xy 126.5 47.9)
       )
     )
@@
       (pts
         (xy 144.9 48.8)
-        (xy 113.7 48.8)
-        (xy 113.7 41.2)
+        (xy 121.2 48.8)
+        (xy 121.2 41.2)
         (xy 144.9 41.2)
       )
@@
         (xy 138.3 85.3)
         (xy 170 85.3)
-        (xy 170 97.5)
-        (xy 113.4 97.5)
+        (xy 170 90.1)
+        (xy 163 90.1)
+        (xy 163 97.5)
+        (xy 120.7 97.5)
+        (xy 120.7 89.7)
+        (xy 120.6 89.6)
+        (xy 113.4 89.6)
         (xy 113.4 73.6)
         (xy 138.3 73.6)
@@
     (polygon
       (pts
+        (xy 162.8 47.7)
+        (xy 171 47.7)
         (xy 171 76.1)
         (xy 143.5 76.1)
         (xy 143.5 41.5)
-        (xy 171 41.5)
+        (xy 162.8 41.5)
       )
     )
