File: PCBs/DolbyDecoder/1.1/DolbyDecoder.kicad_sch (KiCad schematic)
At the start: 93 parts, among them J1 Conn_01x03_Male, J10 Conn_01x04_Male, J11 Conn_01x03_Male, J12 Conn_01x06_Male, J13 Conn_01x04_Male, J2 Conn_01x03_Male, J3 Conn_01x02, J4 Conn_01x04_Male, J5 Conn_01x02_Male, J6 Conn_01x02_Male, J7 Conn_01x02_Male, J8 Conn_01x02_Male, J9 Conn_01x02_Male, U1 AMS1117-2.5, U2 AMS1117-2.5, U3 SPA130, X1 TXC-7C

Commit message: Updated
Parts:
- added R26: 47R, Resistor_SMD:R_0805_2012Metric_Pad1.20x1.40mm_HandSolder, symbol Device:R_Small
- C17: renamed from C4; value 47U -> 10U
- C18: renamed from C1; value 47U -> 10U
- C22: renamed from C7; value 47U -> 10U
- C33: renamed from C17; value 47U -> 10U
- renumbered C2 to C1, C15 to C10, C29 to C11, C28 to C12, C25 to C13, C24 to C14, C31 to C15, C30 to C16, C23 to C19, C6 to C2, C5 to C21, C19 to C23, C13 to C24, C10 to C25, C22 to C26, C16 to C27, C8 to C28, C12 to C29, C26 to C3, C18 to C30, C11 to C31, C3 to C32, C35 to C34, C34 to C35, C27 to C4, C9 to C5, C21 to C6, C14 to C7, C33 to C8, C32 to C9, D3 to D2, D4 to D3, D2 to D4, H4 to H2, H2 to H4, J9 to J1, J3 to J10, J4 to J11, J7 to J12, J5 to J13, J8 to J2, J12 to J3, J6 to J4, J2 to J5, J13 to J6, J1 to J7, J11 to J8, J10 to J9, R5 to R1, R9 to R10, R8 to R11, R7 to R12, R32 to R13, R22 to R14, R31 to R15, R23 to R16, R30 to R17, R29 to R18, R4 to R2, R26 to R20, R15 to R22, R13 to R23, R17 to R24, R16 to R25, R1 to R27, R25 to R28, R28 to R29, R24 to R30, R20 to R31, R2 to R32, R27 to R34, R18 to R4, R14 to R5, R11 to R6, R6 to R7, R12 to R8, R10 to R9, U3 to U1, U1 to U2, U2 to U3
Connections:
- net GND: no longer J6.4 (Pin_4)
- net at U1.72 (PCM_OUT0): now also R26.1
- new net I2S_D4: J6.4 (Pin_4), R26.2
Other:
- moved on the sheet: R4

Commit message: Major updates
Parts:
- C19: value 10N -> 100N
Changed lines of the file:
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@@
       (effects (font (size 1.27 1.27)) (justify left))
     )
-    (property "Value" "10N" (at 53.34 79.375 90)
+    (property "Value" "100N" (at 53.34 79.375 90)
       (effects (font (size 1.27 1.27)) (justify left))
     )
