File: PCBs/Rectifier/1.0/Rectifier.kicad_sch (KiCad schematic)
At the start: 17 parts, among them J1 Conn_01x03_Male, J2 Conn_01x02_Male, J3 Conn_01x02_Male

Commit message: Major updates
Parts:
- R2, R4: value 10R -> 10R 2W
