File: PCBs/Relay AC/1.0/ ACRelay.kicad_pcb (KiCad board)
At the start: 2 copper layers, 25 x 55 mm, 18 parts, among them J1 Conn_01x02_Male, J2 Conn_01x02_Male, J3 Screw_Terminal_01x02, J4 Conn_01x02_Male, J5 Screw_Terminal_01x02, J6 Screw_Terminal_01x02, J7 Screw_Terminal_01x02, Q1 2SC1945

Commit message: Major updates
Parts:
- removed RL1: G2RL-2-ASI-DC5, Relay_THT:Relay_DPDT_Omron_G2RL
- added K1: Relay_DPDT, Relay_THT:Relay_DPDT_Omron_G2RL-2, F.Cu at (151.5, 126.0)
