File: PCBs/Relay AC/1.0/ ACRelay.kicad_sch (KiCad schematic)
At the start: 18 parts, among them J1 Conn_01x02_Male, J2 Conn_01x02_Male, J3 Screw_Terminal_01x02, J4 Conn_01x02_Male, J5 Screw_Terminal_01x02, J6 Screw_Terminal_01x02, J7 Screw_Terminal_01x02, Q1 2SC1945

Commit message: Major updates
Parts:
- removed RL1: G2RL-2-ASI-DC5, Relay_THT:Relay_DPDT_Omron_G2RL, symbol Relay:G2RL-2-ASI-DC5
- added K1: Relay_DPDT, Relay_THT:Relay_DPDT_Omron_G2RL-2, symbol Relay:Relay_DPDT
Connections:
- net 5V: now also K1.A1
- net AC1: now also K1.21
- net AC1OUT: now also K1.14
- net AC2: now also K1.11
- net AC2OUT: now also K1.24
- net at D1.2 (A), Q1.3 (C): now also K1.A2
