File: PCBs/Power Supply (Digital)/1.0/DPSU.kicad_pcb (KiCad board)
At the start: 2 copper layers, 55 x 45 mm, 30 parts, among them J1 Conn_01x02_Male, J2 Conn_01x03_Male, U1 AZ1117-3.3

Commit message: Major updates
Parts:
- PS1: footprint Transformer_THT:HLK-10M05 10W 5V DC -> Components:HLK-10M05
- moved PS1 3.11 mm to (160.0, 95.4)
Routing:
- net AGND: track 65.2 -> 64.5 mm

Commit message: Major updates
Parts:
- D2: value GREEN -> WHITE
- R1: value 30R -> 510R
- R2: value 70R -> 750R
