File: PCBs/Power Supply (Digital)/1.0/DPSU.kicad_sch (KiCad schematic)
At the start: 30 parts, among them J1 Conn_01x02_Male, J2 Conn_01x03_Male, U1 AZ1117-3.3

Commit message: Major updates
Parts:
- PS1: footprint Transformer_THT:HLK-10M05 10W 5V DC -> Components:HLK-10M05

Commit message: Major updates
Parts:
- D2: value GREEN -> WHITE
- R1: value 30R -> 510R
- R2: value 70R -> 750R
Changed lines of the file:
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@@
       (effects (font (size 1.27 1.27)) (justify right))
     )
-    (property "Value" "GREEN" (at 250.317 96.7104 90)
+    (property "Value" "WHITE" (at 250.317 96.7104 90)
       (effects (font (size 1.27 1.27)) (justify right))
     )
@@
       (effects (font (size 1.27 1.27)) (justify left))
     )
-    (property "Value" "30R" (at 249.047 104.1399 0)
+    (property "Value" "510R" (at 249.047 104.1399 0)
       (effects (font (size 1.27 1.27)) (justify left))
     )
@@
       (effects (font (size 1.27 1.27)) (justify left))
     )
-    (property "Value" "70R" (at 236.22 104.2669 0)
-      (effects (font (size 1.27 1.27)) (justify left))
-    )
+    (property "Value" "750R" (at 236.22 104.2669 0)
+      (effects (font (size 1.27 1.27)) (justify left))
+    )
