File: PCBs/Power Supply (Opamps)/1.0/OpampPower.kicad_pcb (KiCad board)
At the start: 2 copper layers, 55 x 45 mm, 30 parts, among them J1 Conn_01x02_Male, J2 Conn_01x02_Male, J3 Conn_01x03_Male, J4 Conn_01x03_Male, J5 Conn_01x03_Male, U1 LM317_SOT-223, U2 LM337_SOT223

Commit message: Major updates
Parts:
- R3, R6: value 220R -> 130R
- R4, R5: value 820R -> 910R
- TR1: value TEZ2.6-D-2 -> 230V 2x9V 2.3VA

Commit message: Major updates
Parts:
- D1: value LED -> BLUE
- D2: value LED -> YELLOW
- R1, R2: value 750R -> 3.3K
- R3, R6: value 130R -> 120R
- R4, R5: value 910R -> 750R
