File: PCBs/Power Supply (Opamps)/1.0/OpampPower.kicad_sch (KiCad schematic)
At the start: 30 parts, among them J1 Conn_01x02_Male, J2 Conn_01x02_Male, J3 Conn_01x03_Male, J4 Conn_01x03_Male, J5 Conn_01x03_Male, U1 LM317_SOT-223, U2 LM337_SOT223

Commit message: Major updates
Parts:
- R3, R6: value 220R -> 130R
- R4, R5: value 820R -> 910R
- TR1: value TEZ2.6-D-2 -> 230V 2x9V 2.3VA

Commit message: Major updates
Parts:
- D1: value LED -> BLUE
- D2: value LED -> YELLOW
- R1, R2: value 750R -> 3.3K
- R3, R6: value 130R -> 120R
- R4, R5: value 910R -> 750R
Changed lines of the file:
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@@
       (effects (font (size 1.27 1.27)) (justify left))
     )
-    (property "Value" "750R" (at 213.36 49.1489 0)
+    (property "Value" "3.3K" (at 213.36 49.1489 0)
       (effects (font (size 1.27 1.27)) (justify left))
     )
@@
       (effects (font (size 1.27 1.27)) (justify left))
     )
-    (property "Value" "130R" (at 154.051 127.6349 0)
+    (property "Value" "120R" (at 154.051 127.6349 0)
       (effects (font (size 1.27 1.27)) (justify left))
     )
@@
       (effects (font (size 1.27 1.27)) (justify left))
     )
-    (property "Value" "910R" (at 149.352 139.7001 0)
+    (property "Value" "750R" (at 149.352 139.7001 0)
       (effects (font (size 1.27 1.27)) (justify left))
     )
@@
       (effects (font (size 1.27 1.27)) (justify right))
     )
-    (property "Value" "LED" (at 225.679 56.9594 90)
+    (property "Value" "BLUE" (at 225.679 56.9594 90)
       (effects (font (size 1.27 1.27)) (justify right))
     )
@@
       (effects (font (size 1.27 1.27)) (justify left))
     )
-    (property "Value" "130R" (at 149.352 148.5901 0)
+    (property "Value" "120R" (at 149.352 148.5901 0)
       (effects (font (size 1.27 1.27)) (justify left))
     )
@@
       (effects (font (size 1.27 1.27)) (justify left))
     )
-    (property "Value" "750R" (at 224.409 49.0219 0)
+    (property "Value" "3.3K" (at 224.409 49.0219 0)
       (effects (font (size 1.27 1.27)) (justify left))
     )
@@
       (effects (font (size 1.27 1.27)) (justify left))
     )
-    (property "Value" "910R" (at 154.051 136.0169 0)
+    (property "Value" "750R" (at 154.051 136.0169 0)
       (effects (font (size 1.27 1.27)) (justify left))
     )
@@
       (effects (font (size 1.27 1.27)) (justify right))
     )
-    (property "Value" "LED" (at 214.63 57.0864 90)
+    (property "Value" "YELLOW" (at 214.63 57.0864 90)
       (effects (font (size 1.27 1.27)) (justify right))
     )
