File: PCBs/Channel Amplifier/1.1/PowerAmp.kicad_sch (KiCad schematic)
At the start: 42 parts, among them J1 Conn_01x02_Male, J2 Conn_01x02_Male, J3 Conn_01x02_Male, J4 Conn_01x02_Male, J5 Conn_01x02_Male, J6 Conn_01x02_Male, J7 Conn_01x03_Male, J8 Conn_01x02_Male, J9 Conn_01x03_Male, U2 TMP100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

Commit message: Major updates
Parts:
- C3, C8: value 47U 50V -> 33U 50V
- Rf1: value 20K -> 23.7K
Changed lines of the file:
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@@
       (effects (font (size 1.27 1.27)))
     )
-    (property "Value" "20K" (at 114.3 153.162 90)
+    (property "Value" "23.7K" (at 114.3 153.162 90)
       (effects (font (size 1.27 1.27)))
     )
@@
       (effects (font (size 1.27 1.27)))
     )
-    (property "Value" "47U 50V" (at 99.7839 80.01 90)
+    (property "Value" "33U 50V" (at 99.7839 80.01 90)
       (effects (font (size 1.27 1.27)))
     )
@@
       (effects (font (size 1.27 1.27)))
     )
-    (property "Value" "47U 50V" (at 100.8761 129.54 90)
-      (effects (font (size 1.27 1.27)))
-    )
+    (property "Value" "33U 50V" (at 100.8761 129.54 90)
+      (effects (font (size 1.27 1.27)))
+    )

Commit message: Updates
Parts:
- C3, C8: value 33U 50V -> 22U 50V
- Ci1: value 1000U 35V -> 1000U 50V
Other:
- moved on the sheet: H1, H2, H3, H4, J2, J8, J9
