File: PCBs/DAC/1.1/DAC.kicad_sch (KiCad schematic)
At the start: 40 parts, among them J1 Conn_01x04_Male, J10 Conn_01x02_Male, J11 Conn_01x02_Male, J12 Conn_01x02_Male, J13 Conn_01x02_Male, J14 Conn_01x02_Male, J15 Conn_01x02_Male, J2 Conn_01x02_Male, J3 Conn_01x04_Male, J4 Conn_01x03_Male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

Commit message: Updates
Parts:
- D1: value YELLOW -> BLUE
Changed lines of the file:
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@@
       (effects (font (size 1.27 1.27)) (justify right))
     )
-    (property "Value" "YELLOW" (at 270.129 144.3354 90)
+    (property "Value" "BLUE" (at 270.129 144.3354 90)
       (effects (font (size 1.27 1.27)) (justify right))
     )
