File: PCBs/DAC/1.2/DAC.kicad_pcb (KiCad board)
At the start: 2 copper layers, 55 x 55 mm, 41 parts, among them J1 Conn_01x04_Male, J10 Conn_01x02_Male, J11 Conn_01x02_Male, J12 Conn_01x02_Male, J13 Conn_01x02_Male, J14 Conn_01x02_Male, J15 Conn_01x02_Male, J16 Conn_01x02_Male, J2 Conn_01x02_Male, J3 Conn_01x04_Male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

Commit message: Dolby Working
Parts:
- added U2: PCM5122PW, Package_SO:TSSOP-28_4.4x9.7mm_P0.65mm, F.Cu at (3.88, 5.12)
