File: PCBs/DolbyDecoder/1.2/DolbyDecoder.kicad_pcb (KiCad board)
At the start: 2 copper layers, 95 x 55 mm, 128 parts, among them J1 Conn_01x02, J2 Conn_01x04_Male, J3 Conn_01x04_Male, J4 Conn_01x02_Male, J5 Conn_01x02_Male, J6 Conn_01x04_Pin, J7 Conn_01x04_Pin, J8 Conn_01x04_Pin, U1 PCM5122PW, U2 PCM5122PW, U3 PCM5122PW, U4 SPA130, U5 AMS1117-2.5, U6 AMS1117-2.5, U7 AMS1117-3.3, X1 TXC-7C

Commit message: Added button debounce code
Parts:
- removed the C48 at (174.1, 56.8)
- added C68: C_Polarized, Capacitor_THT:CP_Radial_D6.3mm_P2.50mm, F.Cu at (205.9, 82.3)
- added C69: C_Polarized, Capacitor_THT:CP_Radial_D6.3mm_P2.50mm, F.Cu at (205.9, 74.2)
- added J4: Conn_01x02, Connector_PinHeader_2.54mm:PinHeader_1x02_P2.54mm_Vertical, F.Cu at (165.7, 87.1)
- added J5: Conn_01x02, Connector_PinHeader_2.54mm:PinHeader_1x02_P2.54mm_Vertical, F.Cu at (158.3, 87.1)
- added J6: Conn_01x02, Connector_PinHeader_2.54mm:PinHeader_1x02_P2.54mm_Vertical, F.Cu at (162.0, 44.6)
- added J9: Conn_01x02, Connector_PinHeader_2.54mm:PinHeader_1x02_P2.54mm_Vertical, F.Cu at (194.3, 56.5)
- added R30: 4.7K, Resistor_SMD:R_0603_1608Metric_Pad0.98x0.95mm_HandSolder, B.Cu at (187.0, 59.3)
- C1, C2, C3, C4, C5, C6: value 2.2n -> 2.2n C0G
- D1: value YELLOW -> BLUE
- D3: value ORANGE -> WHITE
- R16, R18: value 10K -> 4.7K
- R24: renamed from R23; value 160R -> 100R
- R28: renamed from R27; value 160R -> 100R
- X1: moved to B.Cu
- moved J1 23.5 mm to (153.5, 44.9)
- moved J3 23.4 mm to (130.0, 44.9)
- moved C65 6.59 mm to (188.0, 74.4)
- moved C75 5.09 mm to (170.0, 91.2), turned to -90 degrees
- moved C57 1.71 mm to (191.2, 73.7), turned to 90 degrees
- moved C59 1.70 mm to (191.2, 82.4), turned to -90 degrees
- moved C60 1.64 mm to (191.2, 69.1), turned to 90 degrees
- moved C58 1.58 mm to (191.2, 77.9), turned to 90 degrees
- moved R29 1.56 mm to (197.0, 69.2), turned to 90 degrees
- moved R27 1.31 mm to (197.0, 82.4), turned to -90 degrees
- moved R25 1.30 mm to (197.0, 73.7), turned to 90 degrees
- moved R26 1.14 mm to (197.0, 77.9), turned to 90 degrees
- moved C64 0.83 mm to (194.2, 69.2), turned to 90 degrees
- moved C61 0.72 mm to (194.2, 73.7), turned to 90 degrees
- moved C63 0.69 mm to (194.2, 82.4), turned to -90 degrees
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- renumbered C12 to C10, C7 to C11, C13 to C12, C14 to C13, C8 to C14, C49 to C48, C50 to C49, C51 to C50, C52 to C51, C53 to C52, C61 to C53, C55 to C54, C54 to C55, C59 to C56, C56 to C57, C57 to C58, C58 to C59, C62 to C61, C63 to C62, C64 to C63, C65 to C64, C66 to C65, C67 to C66, C68 to C67, C9 to C7, C69 to C70, C70 to C71, C71 to C72, C72 to C73, C73 to C74, C74 to C75, C75 to C76, C10 to C8, C11 to C9, J8 to J1, J3 to J10, J4 to J11, J5 to J12, J7 to J2, J6 to J3, J1 to J7, J2 to J8, R2 to R1, R3 to R2, R29 to R20, R20 to R21, R21 to R22, R22 to R23, R24 to R25, R25 to R26, R26 to R27, R28 to R29, R4 to R3, R5 to R4, R6 to R5, R1 to R6, U2 to U1, U3 to U2, U1 to U3
Connections:
- C71 pad 1: 5VA -> 5V
- U4 pad 52: 3V3 -> 2.5VA
- U5 pad 3: 5VA -> 5V
- X1 pad 1: unconnected-(X1-EN-Pad1) -> Net-(X1-EN)
Routing:
- net 3V3: track 240.1 -> 273.9 mm, vias 12 -> 15
- net PLLSPDIF: track 18.0 -> 48.3 mm, vias 0 -> 4
- net FL: track 41.8 -> 15.0 mm, vias 0 -> 1
- net 2.5VA: track 58.4 -> 83.7 mm, vias 4 -> 7
- net CLKOUT: track 0.00 -> 25.1 mm, vias 0 -> 4
- net FR: track 42.6 -> 20.2 mm, vias 0 -> 1
- net WCLK: track 58.9 -> 79.0 mm, vias 6 -> 9
- net PCMCLK: track 54.5 -> 74.0 mm, vias 6 -> 5
- net GND: track 202.8 -> 219.4 mm, vias 42 -> 41
- net AGND: track 104.4 -> 87.9 mm, vias 21 -> 24
- net I2S_D2: track 26.4 -> 42.1 mm, vias 0 -> 4
- net RR: track 49.2 -> 64.3 mm, vias 0 -> 2
- net CLKIN: track 8.84 -> 23.5 mm, vias 0 -> 2
- net BCLK: track 55.0 -> 68.0 mm, vias 5 -> 7
- net SCL: track 119.2 -> 107.8 mm
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Other:
- board text added: "CLK"
- board text added: "I2C_ADDR"
- board text added: "I2S_TEST"
- board text added: "POWER"
- board text added: "SPDIF"
- board text removed: "DAC_POWER"
