File: PCBs/Channel Selector (Analog)/1.1/ChannelSelector.kicad_sch (KiCad schematic)
At the start: 125 parts, among them J1 Conn_01x03_Pin, J10 Conn_01x02_Pin, J11 Conn_01x02_Male, J12 Conn_01x04_Pin, J13 Conn_01x04_Pin, J14 Conn_01x04_Pin, J15 Conn_01x04_Pin, J16 Conn_01x03_Pin, J17 Conn_01x02_Pin, J18 Conn_01x02_Pin, J2 Conn_01x03_Pin, J3 Conn_01x03_Pin, J4 Conn_01x03_Pin, J5 Conn_01x02_Pin, J6 Conn_01x02_Pin, J7 Conn_01x02_Pin, J8 Conn_01x02_Pin, J9 Conn_01x02_Pin, K1 EC2-5NU, K10 EC2-5NU, K11 EC2-5NU, K12 EC2-5NU, K2 KEMET, K3 EC2-5NU, K4 EC2-5NU, K5 EC2-5NU, K6 EC2-5NU, K7 EC2-5NU, K8 EC2-5NU, K9 EC2-5NU, Q1 BC859, Q10 BC859, Q2 BC859, Q3 BC859, Q4 BC859, Q5 BC859, Q6 BC859, Q7 BC859, Q8 BC859, Q9 BC859, U1 DS1881, U2 TCA9555, U3 OPA2134

Commit message: Mostly working
Parts:
- added J19: Conn_01x02_Pin, Connector_JST:JST_PH_B2B-PH-K_1x02_P2.00mm_Vertical, symbol Connector:Conn_01x02_Pin
Connections:
- net GND: no longer Q1.3 (C), Q10.3 (C), Q2.3 (C), Q3.3 (C), Q4.3 (C), Q5.3 (C), Q7.3 (C), Q8.3 (C), Q9.3 (C)
- new net PGND: J19.1 (Pin_1), Q1.3 (C), Q10.3 (C), Q2.3 (C), Q3.3 (C), Q4.3 (C), Q5.3 (C), Q7.3 (C), Q8.3 (C), Q9.3 (C)
Changed lines of the file:
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@@
     )
   )
-  (global_label "GND" (shape input) (at 63.246 243.84 270) (fields_autoplaced)
+  (global_label "PGND" (shape input) (at 63.246 243.84 270) (fields_autoplaced)
     (effects (font (size 1.27 1.27)) (justify right))
-    (property "Intersheetrefs" "${INTERSHEET_REFS}" (at 63.246 250.6957 90)
+    (property "Intersheetrefs" "${INTERSHEET_REFS}" (at 63.246 251.9657 90)
       (effects (font (size 1.27 1.27)) (justify right) hide)
     )
@@
     )
   )
-  (global_label "GND" (shape input) (at 239.522 64.77 270) (fields_autoplaced)
+  (global_label "PGND" (shape input) (at 239.522 64.77 270) (fields_autoplaced)
     (effects (font (size 1.27 1.27)) (justify right))
-    (property "Intersheetrefs" "${INTERSHEET_REFS}" (at 239.522 71.6257 90)
+    (property "Intersheetrefs" "${INTERSHEET_REFS}" (at 239.522 72.8957 90)
       (effects (font (size 1.27 1.27)) (justify right) hide)
     )
@@
     )
   )
-  (global_label "GND" (shape input) (at 231.394 245.237 270) (fields_autoplaced)
+  (global_label "PGND" (shape input) (at 231.394 245.237 270) (fields_autoplaced)
     (effects (font (size 1.27 1.27)) (justify right))
-    (property "Intersheetrefs" "${INTERSHEET_REFS}" (at 231.394 252.0927 90)
+    (property "Intersheetrefs" "${INTERSHEET_REFS}" (at 231.394 253.3627 90)
       (effects (font (size 1.27 1.27)) (justify right) hide)
     )
@@
     )
   )
+  (global_label "PGND" (shape input) (at 335.661 198.755 0) (fields_autoplaced)
+    (effects (font (size 1.27 1.27)) (justify left))
+    (property "Intersheetrefs" "${INTERSHEET_REFS}" (at 343.7867 198.755 0)
+      (effects (font (size 1.27 1.27)) (justify left) hide)
+    )
+  )
   (global_label "SCL" (shape input) (at 200.279 92.964 180) (fields_autoplaced)
     (effects (font (size 1.27 1.27)) (justify right))
@@
     )
   )
-  (global_label "GND" (shape input) (at 128.524 246.253 270) (fields_autoplaced)
+  (global_label "PGND" (shape input) (at 128.524 246.253 270) (fields_autoplaced)
     (effects (font (size 1.27 1.27)) (justify right))
-    (property "Intersheetrefs" "${INTERSHEET_REFS}" (at 128.524 253.1087 90)
+    (property "Intersheetrefs" "${INTERSHEET_REFS}" (at 128.524 254.3787 90)
       (effects (font (size 1.27 1.27)) (justify right) hide)
     )
@@
     )
   )
-  (global_label "GND" (shape input) (at 49.149 199.136 270) (fields_autoplaced)
+  (global_label "PGND" (shape input) (at 49.149 199.136 270) (fields_autoplaced)
     (effects (font (size 1.27 1.27)) (justify right))
-    (property "Intersheetrefs" "${INTERSHEET_REFS}" (at 49.149 205.9917 90)
+    (property "Intersheetrefs" "${INTERSHEET_REFS}" (at 49.149 207.2617 90)
       (effects (font (size 1.27 1.27)) (justify right) hide)
     )
@@
     )
   )
-  (global_label "GND" (shape input) (at 174.879 64.135 270) (fields_autoplaced)
+  (global_label "PGND" (shape input) (at 174.879 64.135 270) (fields_autoplaced)
     (effects (font (size 1.27 1.27)) (justify right))
-    (property "Intersheetrefs" "${INTERSHEET_REFS}" (at 174.879 70.9907 90)
+    (property "Intersheetrefs" "${INTERSHEET_REFS}" (at 174.879 72.2607 90)
       (effects (font (size 1.27 1.27)) (justify right) hide)
     )
@@
     )
   )
-  (global_label "GND" (shape input) (at 81.915 130.683 270) (fields_autoplaced)
+  (global_label "PGND" (shape input) (at 81.915 130.683 270) (fields_autoplaced)
     (effects (font (size 1.27 1.27)) (justify right))
-    (property "Intersheetrefs" "${INTERSHEET_REFS}" (at 81.915 137.5387 90)
+    (property "Intersheetrefs" "${INTERSHEET_REFS}" (at 81.915 138.8087 90)
       (effects (font (size 1.27 1.27)) (justify right) hide)
     )
@@
     )
   )
-  (global_label "GND" (shape input) (at 61.214 69.088 270) (fields_autoplaced)
+  (global_label "PGND" (shape input) (at 61.214 69.088 270) (fields_autoplaced)
     (effects (font (size 1.27 1.27)) (justify right))
-    (property "Intersheetrefs" "${INTERSHEET_REFS}" (at 61.214 75.9437 90)
+    (property "Intersheetrefs" "${INTERSHEET_REFS}" (at 61.214 77.2137 90)
       (effects (font (size 1.27 1.27)) (justify right) hide)
     )
@@
     )
   )
-  (global_label "GND" (shape input) (at 111.252 64.389 270) (fields_autoplaced)
+  (global_label "PGND" (shape input) (at 111.252 64.389 270) (fields_autoplaced)
     (effects (font (size 1.27 1.27)) (justify right))
-    (property "Intersheetrefs" "${INTERSHEET_REFS}" (at 111.252 71.2447 90)
+    (property "Intersheetrefs" "${INTERSHEET_REFS}" (at 111.252 72.5147 90)
       (effects (font (size 1.27 1.27)) (justify right) hide)
     )
@@
     )
   )
-  (global_label "GND" (shape input) (at 183.388 248.031 270) (fields_autoplaced)
+  (global_label "PGND" (shape input) (at 183.388 248.031 270) (fields_autoplaced)
     (effects (font (size 1.27 1.27)) (justify right))
-    (property "Intersheetrefs" "${INTERSHEET_REFS}" (at 183.388 254.8867 90)
+    (property "Intersheetrefs" "${INTERSHEET_REFS}" (at 183.388 256.1567 90)
       (effects (font (size 1.27 1.27)) (justify right) hide)
     )
@@
         )
       )
+    )
+  )
+  (symbol (lib_id "Connector:Conn_01x02_Pin") (at 330.581 198.755 0) (unit 1)
+    (in_bom yes) (on_board yes) (dnp no) (fields_autoplaced)
+    (property "Reference" "J19" (at 331.216 193.421 0)
+      (effects (font (size 1.27 1.27)))
+    )
+    (property "Value" "Conn_01x02_Pin" (at 331.216 195.961 0)
+      (effects (font (size 1.27 1.27)))
+    )
+    (property "Footprint" "Connector_JST:JST_PH_B2B-PH-K_1x02_P2.00mm_Vertical" (at 330.581 198.755 0)
+      (effects (font (size 1.27 1.27)) hide)
+    )
+    (property "Datasheet" "~" (at 330.581 198.755 0)
+      (effects (font (size 1.27 1.27)) hide)
+    )
+    (pin "1")
+    (pin "2")
+    (instances
+      (project "ChannelSelector"
+        (path "/ad933f83-dd94-4dcc-b4f2-96fd54138c43"
+          (reference "J19") (unit 1)
+        )
+      )
