File: PCBs/Channel Selector/2.1/ChannelSelector.kicad_pcb (KiCad board)
At the start: 2 copper layers, 55 x 55 mm, 83 parts, among them J1 Conn_01x03_Pin, J10 Conn_01x04_Pin, J11 Conn_01x02_Male, J12 Conn_01x04_Pin, J13 CTO, J14 Conn_01x02_Male, J15 Conn_01x02_Male, J17 Conn_01x02_Male, J18 Conn_01x02_Socket, J19 Conn_01x02_Male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

Commit message: Mostly working
Parts:
- R23: value 1K -> 2K
- moved J18 0.19 mm to (159.7, 113.7)
Connections:
- C17 pad 1: 5V -> 9V
- C22 pad 1: 5V -> 9V
- R23 pad 1: 5V -> 9V
- U1 pad 11: 5V -> 9V
Routing:
- net 9V: track 46.7 -> 90.4 mm, vias 5 -> 9
- net 5V: track 42.4 -> 0.00 mm, vias 3 -> 0
- net AGND: track 49.2 -> 43.3 mm
- net 3V3: track 34.0 -> 32.9 mm
- net GND: track 96.9 -> 96.0 mm
- net Net-(J17-Pin_2): track 10.3 -> 9.53 mm
Other:
- board text removed: "5V"
