File: PCBs/Channel Selector/2.1/ChannelSelector.kicad_sch (KiCad schematic)
At the start: 83 parts, among them J1 Conn_01x03_Pin, J10 Conn_01x04_Pin, J11 Conn_01x02_Male, J12 Conn_01x04_Pin, J13 CTO, J14 Conn_01x02_Male, J15 Conn_01x02_Male, J17 Conn_01x02_Male, J18 Conn_01x02_Socket, J19 Conn_01x02_Male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

Commit message: Mostly working
Parts:
- R23: value 1K -> 2K
Connections:
- net 5V: no longer C17.1, C22.1, R23.1, U1.11 (VCC)
- net 9V: now also C17.1, C22.1, R23.1, U1.11 (VCC)
Changed lines of the file:
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@@
     )
   )
-  (global_label "5V" (shape input) (at 187.071 54.864 90) (fields_autoplaced)
+  (global_label "9V" (shape input) (at 187.071 54.864 90) (fields_autoplaced)
     (effects (font (size 1.27 1.27)) (justify left))
     (property "Intersheetrefs" "${INTERSHEET_REFS}" (at 187.071 49.5807 90)
@@
     )
   )
-  (global_label "5V" (shape input) (at 151.257 77.978 90) (fields_autoplaced)
+  (global_label "9V" (shape input) (at 151.257 77.978 90) (fields_autoplaced)
     (effects (font (size 1.27 1.27)) (justify left))
     (property "Intersheetrefs" "${INTERSHEET_REFS}" (at 151.257 72.6947 90)
@@
     )
   )
-  (global_label "5V" (shape input) (at 160.147 51.181 90) (fields_autoplaced)
+  (global_label "9V" (shape input) (at 160.147 51.181 90) (fields_autoplaced)
     (effects (font (size 1.27 1.27)) (justify left))
     (property "Intersheetrefs" "${INTERSHEET_REFS}" (at 160.147 45.8977 90)
@@
   (symbol (lib_id "Device:R_Small") (at 187.071 57.404 0) (unit 1)
     (in_bom yes) (on_board yes) (dnp no)
-    (property "Reference" "R23" (at 183.515 57.404 0)
-      (effects (font (size 1.27 1.27)) (justify left))
-    )
-    (property "Value" "1K" (at 188.722 58.6739 0)
-      (effects (font (size 1.27 1.27)) (justify left))
-    )
+    (property "Reference" "R23" (at 188.849 56.642 0)
+      (effects (font (size 1.27 1.27)) (justify left))
+    )
+    (property "Value" "2K" (at 188.722 58.6739 0)
+      (effects (font (size 1.27 1.27)) (justify left))
+    )
