File: PCBs/DolbyDecoder/2.4/DolbyDecoder.kicad_sch (KiCad schematic)
At the start: 155 parts, among them J1 Conn_01x04_Pin, J10 Conn_01x02, J11 Conn_01x04_Male, J12 Conn_01x02, J13 Conn_01x04_Male, J14 Conn_01x02_Male, J15 Conn_01x02, J16 Conn_01x02_Male, J2 Conn_01x04_Pin, J3 Conn_01x02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

Commit message: Updates
Parts:
- C14, C15, C9: value 10u -> 10u (tie to gnd)
Changed lines of the file:
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@@
       (effects (font (size 1.27 1.27)))
     )
-    (property "Value" "10u" (at 369.8176 155.448 90)
+    (property "Value" "10u (tie to gnd)" (at 369.8176 155.448 90)
       (effects (font (size 1.27 1.27)))
     )
@@
       (effects (font (size 1.27 1.27)))
     )
-    (property "Value" "10u" (at 454.1456 156.21 90)
+    (property "Value" "10u (tie to gnd)" (at 454.1456 156.21 90)
       (effects (font (size 1.27 1.27)))
     )
@@
       (effects (font (size 1.27 1.27)))
     )
-    (property "Value" "10u" (at 534.4096 156.337 90)
+    (property "Value" "10u (tie to gnd)" (at 534.4096 156.337 90)
       (effects (font (size 1.27 1.27)))
     )
