File: PCBs/CS8416 + PCB5122/1.0/CS8416-PCB5122.kicad_pcb (KiCad board)
At the start: 4 copper layers, 95 x 55 mm, 92 parts, among them J1 Conn_01x04_Pin, J10 Conn_01x02_Male, J11 Conn_01x02_Pin, J12 Conn_01x02_Pin, J13 Conn_01x02_Pin, J14 Conn_01x04_Pin, J15 Conn_01x02_Pin, J16 Conn_01x02_Pin, J17 Conn_01x02_Pin, J18 Conn_01x02_Pin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

Commit message: Updates
Parts:
- C5: value 10u -> 0R
Changed lines of the file:
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@@
         (effects (font (size 0.8 0.8) (thickness 0.1)))
     )
-    (fp_text value "10u" (at 0 1.85) (layer "F.Fab")
+    (fp_text value "0R" (at 0 1.85) (layer "F.Fab")
         (effects (font (size 1 1) (thickness 0.15)))
     )
