File: PCBs/CS8416 + PCB5122/1.0/CS8416-PCB5122.kicad_sch (KiCad schematic)
At the start: 92 parts, among them J1 Conn_01x04_Pin, J10 Conn_01x02_Male, J11 Conn_01x02_Pin, J12 Conn_01x02_Pin, J13 Conn_01x02_Pin, J14 Conn_01x04_Pin, J15 Conn_01x02_Pin, J16 Conn_01x02_Pin, J17 Conn_01x02_Pin, J18 Conn_01x02_Pin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

Commit message: Updates
Parts:
- C5: value 10u -> 0R
Changed lines of the file:
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@@
       (effects (font (size 1.27 1.27)) (justify right))
     )
-    (property "Value" "10u" (at 329.4316 115.062 0)
+    (property "Value" "0R" (at 329.4316 115.062 0)
       (effects (font (size 1.27 1.27)) (justify right))
     )
