File: PCBs/2/Power Supply (Channel)/0.1/PowerSupply.kicad_pcb (KiCad board)
At the start: 2 copper layers, 95 x 95 mm, 32 parts, among them J1 Conn_01x02_Male, J10 Conn_01x03_Male, J2 Conn_01x02_Male, J3 Conn_01x03_Male, J4 Conn_01x03_Male, J7 Conn_01x02_Male

Commit message: PCB updates
Parts:
- added C10: 10u, Capacitor_SMD:C_1206_3216Metric_Pad1.33x1.80mm_HandSolder, F.Cu at (159.5, 108.5)
- added C3: 10u, Capacitor_SMD:C_1206_3216Metric_Pad1.33x1.80mm_HandSolder, F.Cu at (160.0, 120.5)
- added C8: 0.1u, Capacitor_SMD:C_0805_2012Metric_Pad1.18x1.45mm_HandSolder, F.Cu at (162.5, 122.5)
- added C9: 0.1u, Capacitor_SMD:C_0805_2012Metric_Pad1.18x1.45mm_HandSolder, F.Cu at (162.0, 110.0)
- added J5: Conn_01x02_Pin, Connector_JST:JST_PH_B2B-PH-K_1x02_P2.00mm_Vertical, F.Cu at (157.5, 135.4)
- added J6: Conn_01x02_Male, Connector_JST:JST_VH_B2P-VH-B_1x02_P3.96mm_Vertical, F.Cu at (147.9, 59.5)
- added J8: Conn_01x02_Male, Connector_JST:JST_PH_B2B-PH-K_1x02_P2.00mm_Vertical, F.Cu at (166.0, 135.4)
- added U1: INA260, Package_SO:TSSOP-16_4.4x5mm_P0.65mm, F.Cu at (167.1, 127.5)
- added U2: INA260, Package_SO:TSSOP-16_4.4x5mm_P0.65mm, F.Cu at (167.1, 114.6)
- J7: value Conn_01x02_Male -> Conn_01x02_Pin; footprint Connector_JST:JST_VH_B2P-VH-B_1x02_P3.96mm_Vertical -> Connector_JST:JST_PH_B2B-PH-K_1x02_P2.00mm_Vertical
- moved J7 60.6 mm to (145.9, 73.5), turned to 90 degrees
- moved R4 43.8 mm to (218.0, 126.6)
- moved R8 43.8 mm to (212.0, 126.6)
- moved J10 30.0 mm to (148.0, 105.9)
- moved J4 30.0 mm to (148.0, 92.0)
- moved C6 25.5 mm to (223.0, 58.0)
- moved C7 25.5 mm to (223.0, 73.0)
- moved F2 14.8 mm to (192.5, 135.7)
- moved R11 14.8 mm to (200.4, 126.4)
- moved D5 14.8 mm to (196.1, 126.4)
- moved D3 14.3 mm to (196.2, 111.3)
- moved R5 14.3 mm to (200.5, 111.3)
- moved F1 14.3 mm to (192.4, 120.8)
- moved R9 7.52 mm to (228.5, 129.0), turned to 180 degrees
- moved R6 5.88 mm to (228.5, 126.5), turned to 180 degrees
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Connections:
- D3 pad 2: VPOUT_FUSE -> VPOUT
- F1 pad 2: VPOUT_FUSE -> VPOUT
- F2 pad 2: VMOUT_FUSE -> VNOUT
- J10 pad 1: VPOUT -> VPOUT_CHAN
- J10 pad 3: VMOUT -> VNOUT
- J3 pad 1: VPOUT_FUSE -> VPOUT_PSU
- J3 pad 3: VMOUT_FUSE -> VNOUT
- J4 pad 1: VPOUT -> VPOUT_CHAN
- J4 pad 3: VMOUT -> VNOUT
- J7 pad 2: RELAY_GND -> PGND
- R11 pad 2: VMOUT_FUSE -> VNOUT
Routing:
- net VM1: track 0.00 -> 173.1 mm, vias 0 -> 2
- net PGND: track 0.00 -> 165.6 mm, vias 0 -> 8
- net VP1: track 0.00 -> 126.7 mm, vias 0 -> 1
- net Net-(C6-Pad2): track 0.00 -> 89.8 mm, vias 0 -> 4
- net VNOUT: track 0.00 -> 73.9 mm, vias 0 -> 2
- net Net-(C7-Pad2): track 0.00 -> 61.4 mm, vias 0 -> 4
- net VNEGNEG: track 0.00 -> 60.4 mm, vias 0 -> 1
- net GND: track 0.00 -> 59.7 mm, vias 0 -> 3
- net VNEG: track 0.00 -> 54.1 mm, vias 0 -> 2
- net VPOSNEG: track 0.00 -> 44.8 mm, vias 0 -> 2
- net 3V3: track 0.00 -> 43.2 mm, vias 0 -> 4
- net VPOUT: track 0.00 -> 31.2 mm
- net SCL: track 0.00 -> 29.9 mm, vias 0 -> 4
- net VPOS: track 0.00 -> 29.5 mm
- net SDA: track 0.00 -> 28.7 mm, vias 0 -> 3
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- added copper zone on B.Cu, net PGND
- added copper zone on F.Cu, net PGND
- added copper zone on B.Cu, net VNOUT
- added copper zone on F.Cu, net VPOUT
- added copper zone on F.Cu, net VPOUT_CHAN
- added copper zone on F.Cu, net VPOUT_PSU
Other:
- board text added: "3V3"
- board text added: "AGND"
- board text added: "CHANNEL_PWR"
- board text added: "I2C"
- board text added: "TO_GND_LIFT"
- board text removed: "FUSED_POWER"
- board text removed: "PGND/REL_GND"
