File: PCBs/2/Power Supply (Dual)/0.1/PowerSupplyDual.kicad_pcb (KiCad board)
At the start: 4 copper layers, 65 x 55 mm, 51 parts, among them J1 Conn_01x03_Male, J10 Conn_01x02_Pin, J12 Conn_01x02_Pin, J13 Conn_01x02_Pin, J14 Conn_01x02_Pin, J15 Conn_01x02_Pin, J2 Conn_01x02_Pin, J3 Conn_01x03_Male, J4 Conn_01x03_Male, J5 Conn_01x03_Male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

Commit message: PCB updates
Parts:
- removed C2, C3: 10U, Capacitor_SMD:C_1206_3216Metric_Pad1.33x1.80mm_HandSolder
- removed D7: BLUE, LED_SMD:LED_0805_2012Metric_Pad1.15x1.40mm_HandSolder
- removed D8: YELLOW, LED_SMD:LED_0805_2012Metric_Pad1.15x1.40mm_HandSolder
- removed R15: 75R, Resistor_SMD:R_0603_1608Metric_Pad0.98x0.95mm_HandSolder
- removed R16: 750R, Resistor_SMD:R_0603_1608Metric_Pad0.98x0.95mm_HandSolder
- added C16: 10U, Capacitor_SMD:C_1206_3216Metric_Pad1.33x1.80mm_HandSolder, F.Cu at (138.3, 90.2)
- added C18: 10U, Capacitor_SMD:C_1206_3216Metric_Pad1.33x1.80mm_HandSolder, F.Cu at (138.3, 108.1)
- added C19: 220u 10V, Capacitor_THT:CP_Radial_D6.3mm_P2.50mm, F.Cu at (119.2, 102.1)
- added C20: 220u 10V, Capacitor_THT:CP_Radial_D6.3mm_P2.50mm, F.Cu at (119.2, 109.4)
- added C21: 100u 50V, Capacitor_THT:CP_Radial_D8.0mm_P3.50mm, F.Cu at (144.5, 97.7)
- added C22: 100u 50V, Capacitor_THT:CP_Radial_D8.0mm_P3.50mm, F.Cu at (144.5, 88.7)
- added C23: 220u 10V, Capacitor_THT:CP_Radial_D6.3mm_P2.50mm, F.Cu at (126.8, 115.2)
- added C24: 220u 10V, Capacitor_THT:CP_Radial_D6.3mm_P2.50mm, F.Cu at (134.6, 115.1)
- added C25: 33nF, Capacitor_SMD:C_1206_3216Metric_Pad1.33x1.80mm_HandSolder, F.Cu at (162.3, 122.0)
- added C26: 0.1u, Capacitor_SMD:C_0805_2012Metric_Pad1.18x1.45mm_HandSolder, F.Cu at (144.7, 114.3)
- added J11: Conn_01x03_Pin, Connector_PinHeader_2.54mm:PinHeader_1x03_P2.54mm_Vertical, F.Cu at (115.1, 118.6)
- added J16: Conn_01x02_Pin, Connector_PinHeader_2.54mm:PinHeader_1x02_P2.54mm_Vertical, F.Cu at (145.0, 81.8)
- added J17: Conn_01x02_Pin, Connector_JST:JST_PH_B2B-PH-K_1x02_P2.00mm_Vertical, F.Cu at (136.5, 129.6)
- added J9: Conn_01x03_Pin, Connector_PinHeader_2.54mm:PinHeader_1x03_P2.54mm_Vertical, F.Cu at (109.0, 123.3)
- added U6: AMS1117-5.0, Package_TO_SOT_SMD:SOT-223-3_TabPin2, F.Cu at (131.6, 90.1)
- added U7: ZLDO1117QG33TA, Package_TO_SOT_SMD:SOT-223-3_TabPin2, F.Cu at (131.6, 108.0)
- C12: value 0.1u -> 10V 470u; footprint Capacitor_SMD:C_0805_2012Metric_Pad1.18x1.45mm_HandSolder -> Capacitor_THT:CP_Radial_D8.0mm_P3.50mm
- C13, C14: value 680u -> 220u 10V; footprint Capacitor_THT:CP_Radial_D8.0mm_P5.00mm -> Capacitor_THT:CP_Radial_D6.3mm_P2.50mm
- J10: value Conn_01x02_Pin -> Conn_01x03_Pin; footprint Connector_PinHeader_2.54mm:PinHeader_1x02_P2.54mm_Vertical -> Connector_PinHeader_2.54mm:PinHeader_1x03_P2.54mm_Vertical
- L1: value 20uH -> 10uH 21mOhm (710-7447707100); footprint Inductor_SMD:L_Taiyo-Yuden_NR-60xx_HandSoldering -> Inductor_SMD:L_Bourns_SRR1208_12.7x12.7mm
- R9: value 60k -> 76.8k
- U4: value LMR50410XDBVR -> TPS62933; footprint Package_TO_SOT_SMD:SOT-23-6_Handsoldering -> Package_TO_SOT_SMD:SOT-583-8
- U5: value AMS1117-3.3 -> ZLDO1117QG33TA
- moved R1 57.3 mm to (111.7, 81.7), turned to 180 degrees
- moved R2 56.5 mm to (111.7, 79.5), turned to 0 degrees
- moved D1 52.2 mm to (115.5, 81.7), turned to 180 degrees
- moved D2 51.3 mm to (115.5, 79.5), turned to 180 degrees
- moved C11 26.1 mm to (162.3, 119.0), turned to 180 degrees
- moved U4 25.3 mm to (156.5, 118.7), turned to 90 degrees
- moved C7 23.9 mm to (158.0, 130.0)
- moved L1 23.0 mm to (159.1, 107.7)
- moved C10 22.0 mm to (154.5, 129.2)
- moved R9 20.2 mm to (148.0, 114.5)
- moved R10 17.6 mm to (151.2, 114.8)
- moved J10 13.3 mm to (104.0, 118.6), turned to 90 degrees
- moved C13 11.1 mm to (119.3, 86.3)
- moved U3 10.9 mm to (131.6, 81.1)
- moved C6 10.9 mm to (156.3, 124.0), turned to 0 degrees
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Connections:
- C1 pad 2: GND -> PGND
- C10 pad 1: AGND -> PGND
- C12 pad 1: Net-(U4-CB) -> 7V
- C12 pad 2: Net-(U4-SW) -> PGND
- C13 pad 1: 3V3 -> 5V_2
- C14 pad 1: 5V -> 5V_1
- C4 pad 2: GND -> PGND
- C5 pad 2: AGND -> PGND
- C6 pad 2: AGND -> PGND
- C7 pad 1: AGND -> PGND
- C8 pad 1: AGND -> PGND
- C9 pad 2: AGND -> PGND
- D1 pad 1: VN -> GND
- D2 pad 1: PGND -> GND
- J10 pad 1: 3V3 -> 3V3_1
- J10 pad 2: 5V -> GND
- J12 pad 2: 3V3 -> 3V3_1
- J13 pad 2: 3V3 -> 3V3_1
- J14 pad 2: 3V3 -> 3V3_2
- J15 pad 2: 3V3 -> 3V3_2
- J2 pad 2: 5V -> 5V_1
- J6 pad 2: 5V -> 5V_2
- J7 pad 2: 5V -> 5V_1
- J8 pad 2: 5V -> 5V_2
- R1 pad 1: PGND -> 3V3_1
- R10 pad 1: FB -> Net-(U4-FB)
- R2 pad 1: VP -> 5V_1
- R4 pad 2: AGND -> PGND
- R5 pad 2: AGND -> PGND
- R9 pad 2: FB -> Net-(U4-FB)
- U3 pad 1: GND -> PGND
- U3 pad 2: 5V -> 5V_1
- U4 pad 1: Net-(U4-CB) -> unconnected-(U4-RT-Pad1)
- U4 pad 2: PGND -> unconnected-(U4-EN-Pad2)
- U4 pad 3: FB -> VP
- U4 pad 4: VP -> PGND
- U4 pad 5: VP -> Net-(U4-SW)
- U4 pad 6: Net-(U4-SW) -> Net-(U4-BST)
- U5 pad 1: GND -> PGND
- U5 pad 2: 3V3 -> 3V3_1
Routing:
- net 5V_1: track 0.00 -> 88.0 mm, vias 0 -> 1
- net VP: track 0.00 -> 87.7 mm, vias 0 -> 4
- net VN: track 0.00 -> 81.2 mm
- net 5V_2: track 0.00 -> 72.4 mm
- net 3V3_1: track 0.00 -> 72.0 mm, vias 0 -> 3
- net 7V: track 0.00 -> 68.6 mm
- net PGND: track 0.00 -> 68.0 mm, vias 0 -> 19
- net DC_POS: track 0.00 -> 67.3 mm, vias 0 -> 3
- net DC_NEG: track 0.00 -> 60.7 mm, vias 0 -> 2
- net 3V3_2: track 0.00 -> 58.4 mm
- net Net-(U4-SW): track 0.00 -> 35.9 mm, vias 0 -> 2
- net Net-(U2-ADJ): track 0.00 -> 14.3 mm
- net Net-(U4-BST): track 0.00 -> 14.0 mm
- net Net-(U1-ADJ): track 0.00 -> 13.5 mm
- net Net-(U4-SS): track 0.00 -> 11.4 mm
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- added copper zone on In1.Cu, net AGND
- added copper zone on In1.Cu, net GND
- added copper zone on B.Cu, net PGND
- added copper zone on F.Cu, net PGND
Other:
- board text added: "AGND"
- board text added: "ANALOG_POWER"
- board text added: "DIG/ANA PSU VERSION 2.0"
- board text added: "GND"
- board text added: "NEG"
- board text added: "POS"
- board text removed: "DC+"
- board text removed: "DC-"
- board text removed: "DUAL POWER VERSION 1.0"
- board text removed: "GNDS"
- board text removed: "PWR"
