File: PCBs/2/Power Supply (Dual)/0.1/PowerSupplyDual.kicad_sch (KiCad schematic)
At the start: 51 parts, among them J1 Conn_01x03_Male, J10 Conn_01x02_Pin, J12 Conn_01x02_Pin, J13 Conn_01x02_Pin, J14 Conn_01x02_Pin, J15 Conn_01x02_Pin, J2 Conn_01x02_Pin, J3 Conn_01x03_Male, J4 Conn_01x03_Male, J5 Conn_01x03_Male, J6 Conn_01x02_Pin, J7 Conn_01x02_Pin, J8 Conn_01x02_Pin, U1 LM317_SOT-223, U2 LM337_SOT223, U3 AMS1117-5.0, U4 LMR50410XDBVR, U5 AMS1117-3.3

Commit message: PCB updates
Parts:
- removed C12: 0.1u, Capacitor_SMD:C_0805_2012Metric_Pad1.18x1.45mm_HandSolder, symbol Device:C_Small
- removed C2, C3: 10U, Capacitor_SMD:C_1206_3216Metric_Pad1.33x1.80mm_HandSolder, symbol Device:C_Polarized_Small
- removed D7: BLUE, LED_SMD:LED_0805_2012Metric_Pad1.15x1.40mm_HandSolder, symbol Device:LED
- removed D8: YELLOW, LED_SMD:LED_0805_2012Metric_Pad1.15x1.40mm_HandSolder, symbol Device:LED
- removed J10: Conn_01x02_Pin, Connector_PinHeader_2.54mm:PinHeader_1x02_P2.54mm_Vertical, symbol Connector:Conn_01x02_Pin
- removed R15: 75R, Resistor_SMD:R_0603_1608Metric_Pad0.98x0.95mm_HandSolder, symbol Device:R_Small
- removed R16: 750R, Resistor_SMD:R_0603_1608Metric_Pad0.98x0.95mm_HandSolder, symbol Device:R_Small
- removed U4: LMR50410XDBVR, Package_TO_SOT_SMD:SOT-23-6_Handsoldering, symbol Components:LMR50410
- added C12: 10V 470u, Capacitor_THT:CP_Radial_D8.0mm_P3.50mm, symbol Device:C_Polarized_Small
- added C16, C18: 10U, Capacitor_SMD:C_1206_3216Metric_Pad1.33x1.80mm_HandSolder, symbol Device:C_Polarized_Small
- added C19, C20, C23, C24: 220u 10V, Capacitor_THT:CP_Radial_D6.3mm_P2.50mm, symbol Device:C_Polarized_Small
- added C21, C22: 100u 50V, Capacitor_THT:CP_Radial_D8.0mm_P3.50mm, symbol Device:C_Polarized_Small
- added C25: 33nF, Capacitor_SMD:C_1206_3216Metric_Pad1.33x1.80mm_HandSolder, symbol Device:C_Polarized_Small
- added C26: 0.1u, Capacitor_SMD:C_0805_2012Metric_Pad1.18x1.45mm_HandSolder, symbol Device:C_Polarized_Small
- added J10, J11, J9: Conn_01x03_Pin, Connector_PinHeader_2.54mm:PinHeader_1x03_P2.54mm_Vertical, symbol Connector:Conn_01x03_Pin
- added J16: Conn_01x02_Pin, Connector_PinHeader_2.54mm:PinHeader_1x02_P2.54mm_Vertical, symbol Connector:Conn_01x02_Pin
- added J17: Conn_01x02_Pin, Connector_JST:JST_PH_B2B-PH-K_1x02_P2.00mm_Vertical, symbol Connector:Conn_01x02_Pin
- added U4: TPS62933, Package_TO_SOT_SMD:SOT-583-8, symbol Regulator_Switching:TPS62933
- added U6: AMS1117-5.0, Package_TO_SOT_SMD:SOT-223-3_TabPin2, symbol Regulator_Linear:AMS1117-5.0
- added U7: ZLDO1117QG33TA, Package_TO_SOT_SMD:SOT-223-3_TabPin2, symbol Regulator_Linear:AMS1117-5.0
- C13, C14: value 680u -> 220u 10V; footprint Capacitor_THT:CP_Radial_D8.0mm_P5.00mm -> Capacitor_THT:CP_Radial_D6.3mm_P2.50mm
- L1: value 20uH -> 10uH 21mOhm (710-7447707100); footprint Inductor_SMD:L_Taiyo-Yuden_NR-60xx_HandSoldering -> Inductor_SMD:L_Bourns_SRR1208_12.7x12.7mm
- R9: value 60k -> 76.8k
- U5: value AMS1117-3.3 -> ZLDO1117QG33TA
Connections:
- net 7V: now also C12.1, C16.1, C18.1, U6.3 (VI), U7.3 (VI)
- net AGND: now also J11.2 (Pin_2), J17.1 (Pin_1), J17.2 (Pin_2); no longer C10.1, C5.2, C6.2, C7.1, C8.1, C9.2, R4.2, R5.2
- net DC_NEG: now also C23.2, J11.1 (Pin_1)
- net DC_POS: now also J11.3 (Pin_3)
- net GND: now also D1.1 (K), D2.1 (K), J10.2 (Pin_2), J16.1 (Pin_1), J9.2 (Pin_2); no longer C1.2, C4.2, U3.1 (GND), U5.1 (GND)
- net PGND: now also C1.2, C10.1, C4.2, C5.2, C6.2, C7.1, C8.1, C9.2, R4.2, R5.2, U3.1 (GND), U5.1 (GND), C12.2, C16.2, C18.2, C19.2, C20.2, C21.1, C22.2, C24.1, C24.2, C25.2, J16.2 (Pin_2), U4.4 (GND), U6.1 (GND), U7.1 (GND); no longer D2.1 (K), R1.1
- net VN: now also C21.2; no longer D1.1 (K)
- net VP: now also C22.1, U4.3 (VIN); no longer R2.1
- net at L1.1: now also C26.2, U4.5 (SW)
- net 3V3 renamed 3V3_1
- net 3V3_1: now also R1.1, C20.1, J10.1 (Pin_1); no longer C13.1, J14.2 (Pin_2), J15.2 (Pin_2)
- net 5V renamed 5V_1
- net 5V_1: now also R2.1, J9.1 (Pin_1); no longer J6.2 (Pin_2), J8.2 (Pin_2)
- net FB: no longer names the net of R10.1, R9.2
- net FB: now also U4.8 (FB)
- new net: C25.1, U4.7 (SS)
- new net: C26.1, U4.6 (BST)
- new net 3V3_2: C19.1, C23.1, J10.3 (Pin_3), J14.2 (Pin_2), J15.2 (Pin_2), U7.2 (VO)
- new net 5V_2: C13.1, J6.2 (Pin_2), J8.2 (Pin_2), J9.3 (Pin_3), U6.2 (VO)
Other:
- moved on the sheet: C1, C4, R10, R9, U3, U5
