File: PCBs/2/CS8416 + PCB5122/2.1/CS8416-PCB5122.kicad_pcb (KiCad board)
At the start: 4 copper layers, 95 x 55 mm, 92 parts, among them J1 Conn_01x04_Pin, J10 Conn_01x02_Male, J11 Conn_01x02_Pin, J12 Conn_01x02_Pin, J13 Conn_01x02_Pin, J14 Conn_01x04_Pin, J15 Conn_01x02_Pin, J16 Conn_01x02_Pin, J17 Conn_01x02_Pin, J18 Conn_01x02_Pin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

Commit message: Updates
Parts:
- C5: value 0R -> 1n; footprint Capacitor_SMD:C_1206_3216Metric_Pad1.33x1.80mm_HandSolder -> Capacitor_SMD:C_0805_2012Metric_Pad1.18x1.45mm_HandSolder
- R17: footprint Resistor_SMD:R_0603_1608Metric_Pad0.98x0.95mm_HandSolder -> Resistor_SMD:R_0805_2012Metric_Pad1.20x1.40mm_HandSolder
- moved C5 60.2 mm to (96.5, 164.0)
- moved R17 0.14 mm to (104.1, 161.0)
Connections:
- C5 pad 2: Net-(U2-VCOM/DEMP) -> 3V3A
- U2 pad 10: Net-(U2-VCOM/DEMP) -> AGND
Routing:
- net Net-(U2-VCOM/DEMP): track 11.2 -> 0.00 mm
- net AGND: track 38.1 -> 45.1 mm, vias 13 -> 12
- net 3V3A: track 158.4 -> 160.7 mm
- added copper zone on F.Cu, net AGND
