File: PCBs/1/Channel Amplifier/2.0/PowerAmp.kicad_sch (KiCad schematic)
At the start: 37 parts, among them J1 Conn_01x02_Male, J2 Conn_01x02_Male, J3 Conn_01x02_Male, J4 Conn_01x03_Male, J5 Conn_01x02_Male, J6 Conn_01x03_Male, U1 LM3886

Commit message: Fixing audio issues, leave TRUNC off and at 24 bits
Parts:
- CSn1: value 220N PP 100V -> 220N PP 100V
