File: PCBs/AURORA/Microprocessor/0.1/uProcessor.kicad_sch (KiCad schematic)
At the start: 66 parts, among them J1 Conn_01x02_Male, J10 Conn_01x02_Male, J11 Conn_01x02_Male, J12 Conn_01x02_Male, J13 Conn_01x03_Pin, J14 Conn_01x04_Pin, J15 Conn_01x04_Pin, J16 Conn_01x02_Male, J17 Conn_01x06_Male, J18 Conn_01x05_Pin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

Commit message: Fixing audio issues, leave TRUNC off and at 24 bits
Parts:
- removed C10, C13: 0.1U, Capacitor_SMD:C_0805_2012Metric_Pad1.18x1.45mm_HandSolder, symbol Device:C_Small
- removed C15, C5: 10U, Capacitor_SMD:C_1206_3216Metric_Pad1.33x1.80mm_HandSolder, symbol Device:C_Small
- removed H5, H6: MountingHole, MountingHole:MountingHole_3.2mm_M3, symbol Mechanical:MountingHole
- removed J11, J22, J4, J5, J6, J7: Conn_01x02_Male, Connector_JST:JST_PH_B2B-PH-K_1x02_P2.00mm_Vertical, symbol Connector:Conn_01x02_Male
- removed U3: TCA9517DR, Package_SO:SOIC-8_3.9x4.9mm_P1.27mm, symbol Interface_LineDriver:TCA9517DR
- added J4, J5: Conn_01x03_Pin, Connector_JST:JST_PH_B3B-PH-K_1x03_P2.00mm_Vertical, symbol Connector:Conn_01x03_Pin
- U1: footprint Espressif:ESP32-WROOM-32UE -> PCM_Espressif:ESP32-WROOM-32E
Connections:
- net EXT2 is gone; now on net POWER_BUTTON: U1.8 (IO32)
- net 3V3: now also J5.2 (Pin_2)
- net GND: now also J4.2 (Pin_2), J5.1 (Pin_1)
- net POWER_BUTTON: no longer U1.10 (IO25)
- net ADC2 renamed IR_RECV
- net IR_RECV: now also J5.3 (Pin_3)
- net CS3310_CS renamed CHANSEL_CS
- net EXT1 renamed DAC_2
- net DAC_2: now also J4.3 (Pin_3)
- new net DAC_1: J4.1 (Pin_1), U1.10 (IO25)
Other:
- moved on the sheet: J8, J9
