File: PCBs/AURORA/Vinyl Pre-amp/0.1/Phono Pre-amp.kicad_sch (KiCad schematic)
At the start: 59 parts, among them J1 Conn_01x02_Pin, J2 Conn_01x03_Male, J3 Conn_01x03_Male, J4 Conn_01x03_Male, J5 Conn_01x03_Male, J6 Conn_01x03_Pin, U1 OPA2134, U2 OPA2134

Commit message: Fixing audio issues, leave TRUNC off and at 24 bits
Parts:
- removed J1: Conn_01x02_Pin, Connector_PinHeader_2.54mm:PinHeader_1x02_P2.54mm_Vertical, symbol Connector:Conn_01x02_Pin
- added J6: Conn_01x03_Male, Connector_JST:JST_PH_B3B-PH-K_1x03_P2.00mm_Vertical, symbol Connector:Conn_01x03_Male
- renumbered C12 to C1, C3 to C10, C1 to C11, C2 to C12, C11 to C2, C8 to C3, C9 to C4, C10 to C5, C7 to C6, C5 to C7, C6 to C8, C4 to C9, CF8 to CF1, CF7 to CF2, CF6 to CF3, CF5 to CF4, CF4 to CF5, CF3 to CF6, CF2 to CF7, CF1 to CF8, J6 to J1, J5 to J2, J2 to J4, J4 to J5, R18 to R1, R9 to R10, R8 to R11, R7 to R12, R6 to R13, R5 to R14, R4 to R15, R1 to R16, R3 to R17, R2 to R18, R17 to R2, R16 to R3, R15 to R4, R14 to R5, R13 to R6, R12 to R7, R11 to R8, R10 to R9, RA2 to RA1, RA1 to RA2, RV2 to RV1, RV1 to RV2, TP4 to TP1, TP3 to TP2, TP1 to TP3, TP2 to TP4, U2 to U1, U1 to U2
Connections:
- net PGND is gone; now on net AGND: J4.2 (Pin_2)
- net AGND: now also J6.2 (Pin_2)
- net V+: now also J6.3 (Pin_3)
- net V-: now also J6.1 (Pin_1)
