File: PCBs/1/CS8416 + PCB5122/1.0/CS8416-PCB5122.kicad_sch (KiCad schematic)
At the start: 92 parts, among them J1 Conn_01x04_Pin, J10 Conn_01x02_Male, J11 Conn_01x02_Pin, J12 Conn_01x02_Pin, J13 Conn_01x02_Pin, J14 Conn_01x04_Pin, J15 Conn_01x02_Pin, J16 Conn_01x02_Pin, J17 Conn_01x02_Pin, J18 Conn_01x02_Pin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

Commit message: Updates
Changed lines of the file:
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@@
+    (stroke (width 0) (type default))
+  )
+  (wire (pts (xy 323.088 83.439) (xy 323.215 83.439))
     (stroke (width 0) (type default))
   )
@@
     (stroke (width 0) (type default))
   )
+  (wire (pts (xy 323.215 83.439) (xy 323.215 88.265))
+    (stroke (width 0) (type default))
+  )
   (wire (pts (xy 178.689 207.772) (xy 179.451 207.772))
     (stroke (width 0) (type default))
@@
     (stroke (width 0) (type default))
   )
-  (wire (pts (xy 323.215 86.233) (xy 323.215 88.265))
+  (wire (pts (xy 323.088 83.185) (xy 323.088 83.439))
     (stroke (width 0) (type default))
   )
@@
     )
   )
-  (global_label "AGND" (shape input) (at 323.215 86.233 90) (fields_autoplaced)
-    (effects (font (size 1.27 1.27)) (justify left))
-    (property "Intersheetrefs" "${INTERSHEET_REFS}" (at 323.215 78.2887 90)
-      (effects (font (size 1.27 1.27)) (justify left) hide)
-    )
+  (global_label "AGND" (shape input) (at 323.088 83.185 90) (fields_autoplaced)
+    (effects (font (size 1.27 1.27)) (justify left))
+    (property "Intersheetrefs" "${INTERSHEET_REFS}" (at 323.088 75.2407 90)
+      (effects (font (size 1.27 1.27)) (justify left) hide)
+    )
