File: PCBs/AURORA/ADC/0.1/ADC.kicad_pcb (KiCad board)
At the start: 4 copper layers, 85 x 55 mm, 40 parts, among them J1 Conn_01x08_Pin, J13 Conn_01x03_Male, J14 Conn_01x02_Male, J2 Conn_01x08_Pin, J3 Conn_01x03_Pin, J4 Conn_01x08_Pin, J5 Conn_01x02_Pin, J6 Conn_01x03_Pin, J7 Conn_01x02_Male, J8 Conn_01x02_Male, U1 ZLDO1117QG33TA, U2 ADG729, U3 ADG729, U5 TAA5212

Commit message: Updates
Parts:
- removed C18: 470u, Capacitor_THT:CP_Radial_D6.3mm_P2.50mm
- removed C19: 1u, Capacitor_SMD:C_1206_3216Metric_Pad1.33x1.80mm_HandSolder
- removed the C3 at (153.9, 81.3)
- removed the C5 at (153.4, 78.9)
- removed the C7 at (107.8, 102.4)
- removed the J1 at (117.4, 112.8)
- removed J13: Conn_01x03_Male, Connector_JST:JST_PH_B3B-PH-K_1x03_P2.00mm_Vertical
- removed the J4 at (96.3, 63.4)
- removed the J5 at (117.8, 91.2)
- removed R10, R8, R9: 22R, Resistor_SMD:R_0805_2012Metric_Pad1.20x1.40mm_HandSolder
- removed R7: 10K, Resistor_SMD:R_0603_1608Metric_Pad0.98x0.95mm_HandSolder
- removed U3: ADG729, Package_SO:TSSOP-16_4.4x5mm_P0.65mm
- removed U5: TAA5212, Package_DFN_QFN:WQFN-24-1EP_4x4mm_P0.5mm_EP2.6x2.6mm_ThermalVias
- added C10: 10u, Capacitor_SMD:C_1206_3216Metric_Pad1.33x1.80mm_HandSolder, F.Cu at (119.5, 86.5)
- added C11: 0.1u, Capacitor_SMD:C_0805_2012Metric_Pad1.18x1.45mm_HandSolder, F.Cu at (119.8, 89.4)
- added C12: 10u, Capacitor_SMD:C_1206_3216Metric_Pad1.33x1.80mm_HandSolder, F.Cu at (128.0, 87.6)
- added C13: 1u, Capacitor_SMD:C_1206_3216Metric_Pad1.33x1.80mm_HandSolder, F.Cu at (120.6, 92.2)
- added C14: 10n C0G, Capacitor_SMD:C_0805_2012Metric_Pad1.18x1.45mm_HandSolder, F.Cu at (126.1, 99.3)
- added C6: 0.1u, Capacitor_SMD:C_0805_2012Metric_Pad1.18x1.45mm_HandSolder, F.Cu at (118.8, 79.0)
- added D1: BLUE, LED_SMD:LED_0805_2012Metric, F.Cu at (168.5, 93.7)
- added J2: Conn_01x02_Male, Connector_JST:JST_PH_B2B-PH-K_1x02_P2.00mm_Vertical, F.Cu at (106.0, 112.7)
- added J6: Conn_01x03_Pin, Connector_JST:JST_PH_B3B-PH-K_1x03_P2.00mm_Vertical, F.Cu at (88.7, 100.9)
- added R3: 75R, Resistor_SMD:R_0603_1608Metric_Pad0.98x0.95mm_HandSolder, F.Cu at (168.5, 97.2)
- added R4: 100R, Resistor_SMD:R_0805_2012Metric_Pad1.20x1.40mm_HandSolder, F.Cu at (122.2, 99.3)
- added R5: 100R, Resistor_SMD:R_0805_2012Metric_Pad1.20x1.40mm_HandSolder, F.Cu at (122.2, 96.8)
- C15: value 10u -> 10u NICHICON 25V; footprint Capacitor_SMD:C_1206_3216Metric_Pad1.33x1.80mm_HandSolder -> Capacitor_THT:CP_Radial_D5.0mm_P2.00mm
- C16: value 0.1u -> 10u NICHICON 25V; footprint Capacitor_SMD:C_0805_2012Metric_Pad1.18x1.45mm_HandSolder -> Capacitor_THT:CP_Radial_D5.0mm_P2.00mm
- C17: value 470u -> 10n C0G; footprint Capacitor_THT:CP_Radial_D6.3mm_P2.50mm -> Capacitor_SMD:C_0805_2012Metric_Pad1.18x1.45mm_HandSolder
- C8: value 0.1u -> 10u; footprint Capacitor_SMD:C_0805_2012Metric_Pad1.18x1.45mm_HandSolder -> Capacitor_SMD:C_1206_3216Metric_Pad1.33x1.80mm_HandSolder
- H1, H2, H3, H4: footprint MountingHole:MountingHole_3.2mm_M3 -> MountingHole:MountingHole_3.2mm_M3_DIN965_Pad_TopOnly
- J1: renamed from J2; value Conn_01x08_Pin -> Conn_01x04_Pin; footprint Connector_JST:JST_PH_B8B-PH-K_1x08_P2.00mm_Vertical -> Connector_JST:JST_PH_B4B-PH-K_1x04_P2.00mm_Vertical
- J8: value Conn_01x02_Male -> Conn_01x03_Pin; footprint Connector_PinHeader_2.54mm:PinHeader_1x02_P2.54mm_Vertical -> Connector_PinHeader_2.54mm:PinHeader_1x03_P2.54mm_Vertical
- R2: value 4.7K -> 22R; footprint Resistor_SMD:R_0603_1608Metric_Pad0.98x0.95mm_HandSolder -> Resistor_SMD:R_0805_2012Metric_Pad1.20x1.40mm_HandSolder
- U2: value ADG729 -> PCM1863; footprint Package_SO:TSSOP-16_4.4x5mm_P0.65mm -> Package_SO:TSSOP-30_4.4x7.8mm_P0.5mm
- moved J8 54.7 mm to (89.1, 79.5), turned to 0 degrees
- moved J1 49.3 mm to (97.4, 63.5)
- moved R1 42.8 mm to (94.8, 79.4), turned to 180 degrees
- moved J7 41.9 mm to (97.3, 112.7)
- moved R2 41.8 mm to (104.5, 71.2), turned to 90 degrees
- moved C17 34.6 mm to (126.1, 96.8), turned to 0 degrees
- moved C5 32.4 mm to (111.5, 79.4)
- moved C15 31.8 mm to (140.7, 104.1), turned to 0 degrees
- moved C16 30.3 mm to (147.2, 104.1), turned to 0 degrees
- moved C7 28.1 mm to (113.8, 81.1)
- moved C8 24.1 mm to (119.4, 81.3)
- moved C3 18.8 mm to (149.6, 83.6), turned to 0 degrees
- moved C9 15.7 mm to (118.9, 84.2)
- moved J3 13.4 mm to (161.0, 105.4), turned to 0 degrees
- moved U2 13.4 mm to (110.8, 88.8), turned to 180 degrees
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- renumbered C13 to C1, C1 to C2, C14 to C3, C2 to C5, C6 to C7, J7 to J3, J6 to J4, J3 to J5, J14 to J7
Connections:
- C15 pad 1: DREG -> LEFT_IN
- C15 pad 2: GND -> Net-(C15-Pad2)
- C16 pad 1: DREG -> RIGHT_IN
- C16 pad 2: GND -> Net-(C16-Pad2)
- C17 pad 1: V+ -> Net-(U2-VINR1)
- C17 pad 2: GND -> AGND
- C9 pad 1: 3V3 -> LDO
- J1 pad 1: GND -> I2S_MCLK_OUT
- J1 pad 2: I2S2_MCLK -> I2S_BCLK_OUT
- J1 pad 3: GND -> I2S_LRCLK_OUT
- J1 pad 4: I2S2_BCLK -> I2S_DATA_OUT
- J8 pad 1: ADC_ADDR -> GPIO0
- J8 pad 2: 3V3 -> I2S_MCLK_OUT
- R1 pad 1: I2S3_MCLK_OUT -> Net-(U2-MOSI/GPIO0/DMIN2)
- R1 pad 2: Net-(U5-GPIO1) -> GPIO0
- R2 pad 1: ADC_ADDR -> Net-(U2-DOUT)
- R2 pad 2: GND -> I2S_DATA_OUT
- U2 pad 1: SCL -> AGND
- U2 pad 10: I2S3_BCLK_OUT -> unconnected-(U2-XI-Pad10)
- U2 pad 11: I2S2_BCLK -> LDO
- U2 pad 12: I2S1_BCLK -> GND
- U2 pad 13: GND -> 3V3
- U2 pad 15: GND -> MCLKI
- U2 pad 16: A0 -> I2S_LRCLK_OUT
- U2 pad 2: GND -> AGND
- U2 pad 3: SDA -> Net-(U2-VINL1)
- U2 pad 4: GND -> Net-(U2-VINR1)
- U2 pad 5: I2S1_MCLK -> unconnected-(U2-MICBIAS-Pad5)
- U2 pad 6: I2S2_MCLK -> VREF
- U2 pad 7: I2S3_MCLK_OUT -> AGND
- U2 pad 8: I2S_MCLK_OUT -> 3V3A
- U2 pad 9: I2S_BCLK_OUT -> unconnected-(U2-XO-Pad9)
Routing:
- net SDA: track 93.9 -> 29.1 mm
- net I2S_LRCLK_OUT: track 0.00 -> 63.7 mm, vias 0 -> 1
- net SCL: track 83.5 -> 29.1 mm, vias 4 -> 0
- net I2S3_MCLK_OUT: track 51.6 -> 0.00 mm
- net I2S1_MCLK: track 51.2 -> 0.00 mm, vias 2 -> 0
- net I2S1_BCLK: track 49.7 -> 0.00 mm, vias 2 -> 0
- net MCLKI: track 0.00 -> 49.2 mm, vias 0 -> 1
- net I2S1_DATA: track 47.7 -> 0.00 mm, vias 2 -> 0
- net I2S3_BCLK_OUT: track 47.7 -> 0.00 mm, vias 2 -> 0
- net I2S3_DATA_OUT: track 42.8 -> 0.00 mm, vias 2 -> 0
- net I2S1_LRCLK: track 41.9 -> 0.00 mm, vias 1 -> 0
- net 3V3: track 152.9 -> 111.2 mm, vias 2 -> 0
- net I2S2_LRCLK: track 36.7 -> 0.00 mm, vias 1 -> 0
- net I2S2_LRCLK_OUT: track 36.6 -> 0.00 mm, vias 1 -> 0
- net Net-(U2-DOUT): track 0.00 -> 36.2 mm
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- added copper zone on F.Cu, net AGND
- added copper zone on B.Cu, net GND
- removed copper zone on B.Cu, net AGND
- removed copper zone on In1.Cu, net AGND
- removed copper zone on F.Cu, net GND
- removed copper zone on In2.Cu, net GND
Other:
- copper layers 4 -> 2
- board text added: "3V3"
- board text added: "CTRL"
- board text added: "GND/AGND"
- board text added: "I2S_CLKS"
- board text added: "I2S_OUT"
- board text added: "MCLKI-MCLKO"
- board text removed: "ANALOG_PWR"
- board text removed: "I2S_1"
- board text removed: "I2S_2"
