File: PCBs/AURORA/ADC/0.1/ADC.kicad_sch (KiCad schematic)
At the start: 40 parts, among them J1 Conn_01x08_Pin, J14 Conn_01x02_Male, J2 Conn_01x08_Pin, J3 Conn_01x03_Pin, J4 Conn_01x03_Male, J4 Conn_01x08_Pin, J5 Conn_01x02_Pin, J6 Conn_01x03_Pin, J7 Conn_01x02_Male, J8 Conn_01x02_Male, U1 ZLDO1117QG33TA, U2 ADG729, U3 ADG729, U5 TAA5212

Commit message: Updates
Parts:
- removed C17, C18: 470u, Capacitor_THT:CP_Radial_D6.3mm_P2.50mm, symbol Device:C_Polarized_Small
- removed C19: 1u, Capacitor_SMD:C_1206_3216Metric_Pad1.33x1.80mm_HandSolder, symbol Device:C_Small
- removed C3, C7: 10u, Capacitor_SMD:C_1206_3216Metric_Pad1.33x1.80mm_HandSolder, symbol Device:C_Small
- removed C5: 0.1u, Capacitor_SMD:C_0805_2012Metric_Pad1.18x1.45mm_HandSolder, symbol Device:C_Small
- removed J1, J2, J4: Conn_01x08_Pin, Connector_JST:JST_PH_B8B-PH-K_1x08_P2.00mm_Vertical, symbol Connector:Conn_01x08_Pin
- removed J4: Conn_01x03_Male, Connector_JST:JST_PH_B3B-PH-K_1x03_P2.00mm_Vertical, symbol Connector:Conn_01x03_Male
- removed J5: Conn_01x02_Pin, Connector_PinHeader_2.54mm:PinHeader_1x02_P2.54mm_Vertical, symbol Connector:Conn_01x02_Pin
- removed J8: Conn_01x02_Male, Connector_PinHeader_2.54mm:PinHeader_1x02_P2.54mm_Vertical, symbol Connector:Conn_01x02_Male
- removed R10, R8, R9: 22R, Resistor_SMD:R_0805_2012Metric_Pad1.20x1.40mm_HandSolder, symbol Device:R_Small
- removed R7: 10K, Resistor_SMD:R_0603_1608Metric_Pad0.98x0.95mm_HandSolder, symbol Device:R_Small
- removed U2, U3: ADG729, Package_SO:TSSOP-16_4.4x5mm_P0.65mm, symbol Analog_Switch:ADG729
- removed U5: TAA5212, Package_DFN_QFN:WQFN-24-1EP_4x4mm_P0.5mm_EP2.6x2.6mm_ThermalVias, symbol Custom:TAA5212
- added C10, C12: 10u, Capacitor_SMD:C_1206_3216Metric_Pad1.33x1.80mm_HandSolder, symbol Device:C_Small
- added C11, C6: 0.1u, Capacitor_SMD:C_0805_2012Metric_Pad1.18x1.45mm_HandSolder, symbol Device:C_Small
- added C13: 1u, Capacitor_SMD:C_1206_3216Metric_Pad1.33x1.80mm_HandSolder, symbol Device:C_Small
- added C14, C17: 10n C0G, Capacitor_SMD:C_0805_2012Metric_Pad1.18x1.45mm_HandSolder, symbol Device:C_Small
- added D1: BLUE, LED_SMD:LED_0805_2012Metric, symbol Device:LED
- added J1: Conn_01x04_Pin, Connector_JST:JST_PH_B4B-PH-K_1x04_P2.00mm_Vertical, symbol Connector:Conn_01x04_Pin
- added J2: Conn_01x02_Male, Connector_JST:JST_PH_B2B-PH-K_1x02_P2.00mm_Vertical, symbol Connector:Conn_01x02_Male
- added J6: Conn_01x03_Pin, Connector_JST:JST_PH_B3B-PH-K_1x03_P2.00mm_Vertical, symbol Connector:Conn_01x03_Pin
- added J8: Conn_01x03_Pin, Connector_PinHeader_2.54mm:PinHeader_1x03_P2.54mm_Vertical, symbol Connector:Conn_01x03_Pin
- added R3: 75R, Resistor_SMD:R_0603_1608Metric_Pad0.98x0.95mm_HandSolder, symbol Device:R_Small
- added R4, R5: 100R, Resistor_SMD:R_0805_2012Metric_Pad1.20x1.40mm_HandSolder, symbol Device:R_Small
- added U2: PCM1863, Package_SO:TSSOP-30_4.4x7.8mm_P0.5mm, symbol Custom:PCM1863
- added U3: ~, symbol Custom:PCM1865
- C15: value 10u -> 10u NICHICON 25V; footprint Capacitor_SMD:C_1206_3216Metric_Pad1.33x1.80mm_HandSolder -> Capacitor_THT:CP_Radial_D5.0mm_P2.00mm
- C16: value 0.1u -> 10u NICHICON 25V; footprint Capacitor_SMD:C_0805_2012Metric_Pad1.18x1.45mm_HandSolder -> Capacitor_THT:CP_Radial_D5.0mm_P2.00mm
- C8: value 0.1u -> 10u; footprint Capacitor_SMD:C_0805_2012Metric_Pad1.18x1.45mm_HandSolder -> Capacitor_SMD:C_1206_3216Metric_Pad1.33x1.80mm_HandSolder
- H1, H2, H3, H4: footprint MountingHole:MountingHole_3.2mm_M3 -> MountingHole:MountingHole_3.2mm_M3_DIN965_Pad_TopOnly
- R1: Mouser (none) -> 603-RT0805FRE0722RL
- R2: value 4.7K -> 22R; footprint Resistor_SMD:R_0603_1608Metric_Pad0.98x0.95mm_HandSolder -> Resistor_SMD:R_0805_2012Metric_Pad1.20x1.40mm_HandSolder; Mouser (none) -> 603-RT0805FRE0722RL
- renumbered C13 to C1, C1 to C2, C14 to C3, C2 to C5, C6 to C7, J7 to J3, J6 to J4, J3 to J5, J14 to J7
Connections:
- net 3V3: now also C6.1, R3.2, U2.13 (DVDD), U2.14 (IOVDD); no longer C9.1
- net 3V3A: now also C11.1, C12.1, U2.8 (AVDD)
- net AGND: now also C14.1, C17.2, U2.1 (VINL2), U2.2 (VINR2), U2.27 (VINL4), U2.28 (VINR4), U2.29 (VINL3), U2.30 (VINR3), U2.7 (AGND)
- net GND: now also C10.2, C11.2, C12.2, C13.2, C6.2, D1.1 (K), U2.12 (DGND), U2.25 (MS/AD), U2.26 (MD0); no longer C15.2, C16.2, R2.2
- net I2S_BCLK_OUT: now also J1.2 (Pin_2), J6.2 (Pin_2), U2.17 (BCLK)
- net I2S_DATA_OUT: now also R2.2, J1.4 (Pin_4)
- net I2S_MCLK_OUT: now also J1.1 (Pin_1), J8.2 (Pin_2)
- net LEFT_IN: now also C15.1
- net RIGHT_IN: now also C16.1
- net SCL: now also U2.24 (MC/SCL)
- net SDA: now also U2.23 (MOSI/SDA)
- net VREF: now also C13.1, U2.6 (VREF)
- net GPIO0: now reaches R1.2
- net GPIO0: now also J8.1 (Pin_1)
- net ADC_ADDR: no longer names the net of R2.1
- net ADC_ADDR: now also U2.18 (DOUT)
- removed net DREG: C15.1, C16.1
- net I2S3_MCLK_OUT: no longer names the net of R1.1
- net I2S3_MCLK_OUT: now also U2.22 (MOSI/GPIO0/DMIN2)
- new net: C14.2, R4.2, U2.3 (VINL1)
- new net: C16.2, R5.1
- new net: C17.1, R5.2, U2.4 (VINR1)
- new net: D1.2 (A), R3.1
- new net: C15.2, R4.1
- new net GPIO1: J2.1 (Pin_1), U2.21 (GPIO1/INTA/DMI)
- new net I2S_LRCLK_OUT: J1.3 (Pin_3), J6.3 (Pin_3), U2.16 (LRCLK)
- new net INT: J2.2 (Pin_2), U2.19 (GPIO3/INTC), U2.20 (GPIO2/INTB/DMCLK)
- new net LDO: C10.1, C9.1, U2.11 (LDO)
- new net MCLKI: J6.1 (Pin_1), J8.3 (Pin_3), U2.15 (SCLKI)
Other:
- note removed: "ADG729"
