File: PCBs/AURORA/SPDIF/WM8805/0.1/SPDIF.kicad_pcb (KiCad board)
At the start: 4 copper layers, 85 x 55 mm, 68 parts, among them J1 Conn_01x02_Male, J10 Conn_01x02_Pin, J11 Conn_01x02_Pin, J12 Conn_01x02_Male, J13 Conn_01x02_Male, J14 Conn_02x10_Odd_Even, J2 Conn_01x02_Male, J3 Conn_01x02_Male, J4 CHANSEL, J5 Conn_01x02_Pin, J6 Conn_01x02_Pin, J7 Conn_01x02_Pin, J8 Conn_01x02_Pin, J9 Conn_01x02_Pin, T1 DA101C, T2 DA101C, T3 DA101C, T4 DA101C, U1 ZLDO1117QG33TA, U2 CS8416-xZZ, U3 WM8731SEDS, X1 DFA-S3

Commit message: Updates
Parts:
- removed C15, C18: 0.01u, Capacitor_SMD:C_0805_2012Metric
- removed C16: 10u, Capacitor_SMD:C_1206_3216Metric_Pad1.33x1.80mm_HandSolder
- removed the C3 at (79.3, 37.1)
- removed the C5 at (64.2, 38.2)
- removed the C8 at (68.2, 47.0)
- removed the D1 at (56.0, 32.8)
- removed J14: Conn_02x10_Odd_Even, Connector_PinHeader_2.54mm:PinHeader_2x10_P2.54mm_Vertical
- removed the J3 at (40.3, 30.7)
- removed the J9 at (73.6, 67.9)
- removed the R13 at (90.9, 68.0)
- removed the R7 at (97.8, 61.8)
- removed the R8 at (61.0, 67.8)
- removed the R9 at (70.7, 67.8)
- removed T1, T2, T3, T4: DA101C, Custom:DA101C
- removed TP1, TP2, TP3, TP4: TestPoint, TestPoint:TestPoint_THTPad_2.0x2.0mm_Drill1.0mm
- removed the U1 at (66.6, 32.5)
- removed X1: DFA-S3, Oscillator:Oscillator_SMD_EuroQuartz_XO53-4Pin_5.0x3.2mm_HandSoldering
- added J12: Conn_01x02_Pin, Connector_JST:JST_XH_B2B-XH-A_1x02_P2.50mm_Vertical, F.Cu at (30.3, 72.2)
- added J20: Conn_01x03_Pin, Connector_JST:JST_PH_B3B-PH-K_1x03_P2.00mm_Vertical, F.Cu at (107.9, 65.0)
- added J21: Conn_01x03_Pin, Connector_JST:JST_PH_B3B-PH-K_1x03_P2.00mm_Vertical, F.Cu at (108.0, 74.3)
- added J5: Conn_01x04_Pin, Connector_PinHeader_2.54mm:PinHeader_1x04_P2.54mm_Vertical, F.Cu at (72.0, 31.3)
- added R11: 4.7K, Resistor_SMD:R_0603_1608Metric_Pad0.98x0.95mm_HandSolder, F.Cu at (77.7, 64.3)
- added R14: 75R, Resistor_SMD:R_0603_1608Metric_Pad0.98x0.95mm_HandSolder, F.Cu at (52.2, 75.7)
- added U2: DA101C_C6931652, easyeda2kicad:XFMR-TH_4P-L9.5-W9.0-P5.08-LS10.2_C9900096976, F.Cu at (42.1, 34.5)
- added U4: DA101C_C6931652, easyeda2kicad:XFMR-TH_4P-L9.5-W9.0-P5.08-LS10.2_C9900096976, F.Cu at (42.2, 55.8)
- added U5: DA101C_C6931652, easyeda2kicad:XFMR-TH_4P-L9.5-W9.0-P5.08-LS10.2_C9900096976, F.Cu at (42.2, 66.4)
- added U6: DA101C_C6931652, easyeda2kicad:XFMR-TH_4P-L9.5-W9.0-P5.08-LS10.2_C9900096976, F.Cu at (42.2, 77.0)
- added Y1: 12MHz 3.2x2.5, Crystal:Crystal_SMD_SeikoEpson_FA238-4Pin_3.2x2.5mm, F.Cu at (91.0, 54.0)
- C10: value 0.01u -> 0.1u; footprint Capacitor_SMD:C_1206_3216Metric_Pad1.33x1.80mm_HandSolder -> Capacitor_SMD:C_0805_2012Metric_Pad1.18x1.45mm_HandSolder
- C11: value 0.01u -> 10u; footprint Capacitor_SMD:C_0805_2012Metric -> Capacitor_SMD:C_1206_3216Metric_Pad1.33x1.80mm_HandSolder
- C12: value 22n C0G -> 10u; footprint Capacitor_SMD:C_0805_2012Metric_Pad1.18x1.45mm_HandSolder -> Capacitor_SMD:C_1206_3216Metric_Pad1.33x1.80mm_HandSolder
- C13: value 1n C0G -> 0.01u
- C2: renamed from C7; value 0.01u -> 0.01u C0G
- C4: renamed from C14; value 0.01u -> 0.01u C0G
- C5: renamed from C17; value 0.01u -> 0.01u C0G
- C6: renamed from C4; value 0.01u -> 12p C0G
- C7: renamed from C6; value 10u -> 12p C0G; footprint Capacitor_SMD:C_1206_3216Metric_Pad1.33x1.80mm_HandSolder -> Capacitor_SMD:C_0805_2012Metric_Pad1.18x1.45mm_HandSolder
- C8: renamed from C19; value 0.01u -> 0.01u C0G
- C9: value 10u -> 0.1u; footprint Capacitor_SMD:C_1206_3216Metric_Pad1.33x1.80mm_HandSolder -> Capacitor_SMD:C_0805_2012Metric_Pad1.18x1.45mm_HandSolder
- H1, H2, H3, H4: footprint MountingHole:MountingHole_3.2mm_M3 -> MountingHole:MountingHole_3.2mm_M3_DIN965_Pad_TopOnly
- J1: value Conn_01x02_Male -> Conn_01x04_Pin; footprint Connector_JST:JST_PH_B2B-PH-K_1x02_P2.00mm_Vertical -> Connector_JST:JST_PH_B4B-PH-K_1x04_P2.00mm_Vertical
- J11: footprint Connector_PinHeader_2.54mm:PinHeader_1x02_P2.54mm_Vertical -> Connector_JST:JST_PH_B2B-PH-K_1x02_P2.00mm_Vertical
- J2: value Conn_01x02_Male -> Conn_01x02_Pin; footprint Connector_JST:JST_PH_B2B-PH-K_1x02_P2.00mm_Vertical -> Connector_PinHeader_2.54mm:PinHeader_1x02_P2.54mm_Vertical
- J4: value CHANSEL -> Conn_01x03_Pin; footprint Connector_JST:JST_XH_B4B-XH-A_1x04_P2.50mm_Vertical -> Connector_JST:JST_PH_B3B-PH-K_1x03_P2.00mm_Vertical
- R12: value 22R -> 4.7K; footprint Resistor_SMD:R_1206_3216Metric_Pad1.30x1.75mm_HandSolder -> Resistor_SMD:R_0603_1608Metric_Pad0.98x0.95mm_HandSolder
- R2: renamed from R11; footprint Resistor_SMD:R_1206_3216Metric_Pad1.30x1.75mm_HandSolder -> Resistor_SMD:R_0805_2012Metric_Pad1.20x1.40mm_HandSolder
- R3: renamed from R14; footprint Resistor_SMD:R_1206_3216Metric_Pad1.30x1.75mm_HandSolder -> Resistor_SMD:R_0805_2012Metric_Pad1.20x1.40mm_HandSolder
- R4: value 3K -> 22R
- R5: value 75R -> 22R; footprint Resistor_SMD:R_0603_1608Metric_Pad0.98x0.95mm_HandSolder -> Resistor_SMD:R_0805_2012Metric_Pad1.20x1.40mm_HandSolder
- U1: renamed from U2; value CS8416-xZZ -> WM8805; footprint Package_SO:TSSOP-28_4.4x9.7mm_P0.65mm -> Package_SO:SSOP-28_5.3x10.2mm_P0.65mm
- U3: value WM8731SEDS -> DA101C_C6931652; footprint Package_SO:SSOP-28_5.3x10.2mm_P0.65mm -> easyeda2kicad:XFMR-TH_4P-L9.5-W9.0-P5.08-LS10.2_C9900096976
- moved R13 62.7 mm to (83.3, 74.3), turned to -90 degrees
- moved U3 54.5 mm to (42.2, 45.1)
- moved J17 39.3 mm to (89.6, 79.8), turned to 0 degrees
- moved J8 35.6 mm to (99.4, 65.0), turned to -90 degrees
- moved R5 35.3 mm to (86.8, 39.5), turned to 90 degrees
- moved J10 32.5 mm to (89.6, 73.6), turned to 0 degrees
- moved R3 31.8 mm to (79.6, 39.5), turned to 90 degrees
- moved R2 30.1 mm to (76.0, 39.5), turned to 90 degrees
- moved C13 28.8 mm to (52.2, 71.2)
- moved C9 25.3 mm to (70.5, 62.8), turned to 90 degrees
- moved C7 24.7 mm to (92.2, 58.3), turned to 0 degrees
- moved C6 21.5 mm to (92.4, 49.9), turned to 180 degrees
- moved C12 21.3 mm to (88.0, 63.4), turned to 90 degrees
- moved C10 20.5 mm to (85.3, 62.8)
- moved C11 20.3 mm to (73.1, 63.4), turned to 90 degrees
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- renumbered C2 to C1, C1 to C3, D2 to D1, D3 to D2, J13 to J10, J12 to J17, J5 to J3, J10 to J9, R2 to R1, R1 to R13, R3 to R6, R6 to R7, R15 to R8, R16 to R9
Connections:
- C10 pad 1: AGND -> GND
- C10 pad 2: 3V3A -> 3V3
- C11 pad 2: 3V3 -> 5V
- C12 pad 1: AGND -> GND
- C12 pad 2: Net-(C12-Pad2) -> 3V3
- C13 pad 1: AGND -> SPDIF_5
- C13 pad 2: FILT -> Net-(C13-Pad2)
- C4 pad 2: Net-(T2-SB) -> Net-(C4-Pad2)
- C6 pad 1: AGND -> Net-(U1-XIN)
- C6 pad 2: Net-(U2-RXN) -> AGND
- C7 pad 1: 3V3A -> Net-(U1-XOP)
- C9 pad 2: 3V3 -> 5V
- J1 pad 1: GND -> I2S_SCLK
- J1 pad 2: GPO1 -> I2S_BCLK
- J11 pad 1: GND -> INT
- J11 pad 2: OMCK -> RESET
- J2 pad 2: GPO0 -> AGND
- J4 pad 1: unconnected-(J4-Pin_1-Pad1) -> 3V3
- J4 pad 2: 3V3 -> GND
- J4 pad 3: GND -> 5V
- J8 pad 1: Net-(J8-Pin_1) -> ADDR
- R12 pad 1: Net-(U2-OSCLK) -> ADDR
- R12 pad 2: I2S_BCLK -> GND
- R2 pad 1: Net-(U2-RMCK) -> MCLK_OUT
- R3 pad 1: Net-(U2-SDOUT) -> Net-(U1-BCLK)
- R3 pad 2: I2S_DATA -> I2S_BCLK
- R4 pad 1: FILT -> Net-(U1-LRCLK)
- R4 pad 2: Net-(C12-Pad2) -> I2S_LRCLK
- R5 pad 1: GND -> Net-(U1-DOUT)
- R5 pad 2: Net-(D1-K) (its old number) -> I2S_DATA
- R6 pad 1: Net-(T2-SB) -> Net-(C4-Pad2)
- U1 pad 1: SPDIF_4 -> 5V
- U1 pad 10: AGND -> RESET
- U1 pad 11: AGND -> 3V3
- U1 pad 12: AGND -> GND
- U1 pad 13: AGND -> unconnected-(U1-CLKOUT-Pad13)
- U1 pad 14: GND -> Net-(U1-XOP)
- U1 pad 15: Net-(J9-Pin_1) -> Net-(U1-XIN)
- U1 pad 16: SCL -> Net-(U1-DOUT)
- U1 pad 17: SDA -> DIN
- U1 pad 18: Net-(J8-Pin_1) -> Net-(U1-BCLK)
- U1 pad 19: GPO1 -> Net-(U1-LRCLK)
- U1 pad 2: SPDIF_3 -> SPDIF_2
- U1 pad 20: GPO0 -> MCLK_OUT
- U1 pad 21: 3V3 -> SPDIF_OUT
- U1 pad 22: GND -> AGND
- U1 pad 23: 3V3 -> AGND
- U1 pad 24: Net-(U2-RMCK) -> AGND
- U1 pad 25: OMCK -> SPDIF_5
- U1 pad 26: Net-(U2-SDOUT) -> SPDIF_4
- U1 pad 27: Net-(U2-OSCLK) -> SPDIF_3
- U1 pad 28: Net-(U2-OLRCK) -> GND
- U1 pad 3: SPDIF_2 -> SPDIF_1
- U1 pad 4: SPDIF_1 -> SCL
- U1 pad 5: Net-(U2-RXN) -> NONAUDIO
- U1 pad 6: 3V3A -> UNLOCK
- U1 pad 7: AGND -> SDA
- U1 pad 8: FILT -> INT
- U1 pad 9: RESET -> ADDR
- U3 pad 1: unconnected-(U3-DBVDD-Pad1) -> SPDIF2_IN
- U3 pad 3: unconnected-(U3-BCLK-Pad3) -> SPDIF2_GND
- U3 pad 4: unconnected-(U3-DACDAT-Pad4) -> AGND
- U3 pad 6: unconnected-(U3-ADCDAT-Pad6) -> Net-(C4-Pad2)
Routing:
- net I2S_LRCLK: track 0.00 -> 78.7 mm, vias 0 -> 1
- net I2S_BCLK: track 0.00 -> 72.0 mm, vias 0 -> 1
- net 3V3: track 0.00 -> 68.5 mm
- net I2S_SCLK: track 0.00 -> 68.2 mm, vias 0 -> 1
- net 5V: track 0.00 -> 63.9 mm, vias 0 -> 2
- net AGND: track 0.00 -> 42.2 mm, vias 0 -> 4
- net ADDR: track 0.00 -> 36.0 mm, vias 0 -> 2
- net SPDIF_1: track 0.00 -> 35.1 mm, vias 0 -> 2
- net SPDIF_5: track 0.00 -> 33.9 mm
- net SPDIF_2: track 0.00 -> 32.2 mm, vias 0 -> 2
- net I2S_DATA: track 0.00 -> 29.8 mm
- net SCL: track 0.00 -> 29.6 mm, vias 0 -> 2
- net SPDIF_4: track 0.00 -> 29.5 mm
- net SDA: track 0.00 -> 28.4 mm
- net RESET: track 0.00 -> 27.6 mm, vias 0 -> 2
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- added copper zone on B.Cu, net AGND
- added copper zone on In1.Cu, net AGND
- added copper zone on F.Cu, net GND
- added copper zone on In2.Cu, net GND
Other:
- board text added: "CTRL"
- board text added: "GND/AGD"
- board text added: "I2C_ADDR"
- board text added: "I2S_CLKS"
- board text added: "I2S_OUT"
- board text added: "SPDIF5"
- board text removed: "3V3A"
- board text removed: "GND"
- board text removed: "GPO2"
- board text removed: "OMCK"
- board text removed: "RESET"
- board text removed: "SPDIF_AD1"
- board text removed: "SPDIF_AD2"
