File: PCBs/AURORA/DAC/1.0/DAC.kicad_pcb (KiCad board)
At the start: 2 copper layers, 85 x 55 mm, 67 parts, among them J1 Conn_01x03_Pin, J10 Conn_01x02_Pin, J2 Conn_01x03_Pin, J3 Conn_01x03_Pin, J4 Conn_01x02_Pin, J5 Conn_01x03_Pin, J6 Conn_01x02_Pin, J7 Conn_01x04_Pin, J8 Conn_01x04_Pin, J9 Conn_01x04_Pin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

Commit message: Moving files
Parts:
- removed J10: Conn_01x02_Pin, Connector_JST:JST_PH_B2B-PH-K_1x02_P2.00mm_Vertical
- added J11: Conn_01x03_Pin, Connector_JST:JST_PH_B3B-PH-K_1x03_P2.00mm_Vertical, F.Cu at (122.2, 109.2)
- moved J9 3.20 mm to (107.1, 109.2)
- moved J8 2.16 mm to (87.1, 109.2)
- moved C29 1.88 mm to (73.1, 95.9)
- moved C36 1.88 mm to (73.8, 98.6)
- moved C2 1.70 mm to (70.9, 68.8)
- moved C1 1.70 mm to (68.6, 68.8)
- moved R1 1.70 mm to (68.6, 72.9)
- moved R2 1.70 mm to (70.9, 72.9)
- moved J7 1.12 mm to (67.1, 109.2)
Connections:
- U3 pad 25: unconnected-(U3-XSMT-Pad25) -> XSMT
- U4 pad 25: unconnected-(U4-XSMT-Pad25) -> XSMT
- U5 pad 25: unconnected-(U5-XSMT-Pad25) -> XSMT
Routing:
- net XSMT: track 0.00 -> 72.0 mm, vias 0 -> 5
- net AGND: track 30.9 -> 15.6 mm, vias 13 -> 9
- net GND: track 2.72 -> 0.00 mm
- net 3V3: track 141.9 -> 139.7 mm, vias 1 -> 8
- net SDA: track 79.5 -> 81.3 mm, vias 1 -> 10
- net 3V3A: track 114.9 -> 116.6 mm, vias 0 -> 7
- net SCL: track 77.0 -> 78.5 mm
- net LRCLK2: track 18.3 -> 17.0 mm, vias 1 -> 0
- net BCLK2: track 18.1 -> 16.7 mm
- net DATA2: track 19.4 -> 18.2 mm, vias 0 -> 1
- net LW_OUT_PRE: track 12.5 -> 13.7 mm
- net Net-(U4-LDOO): track 6.34 -> 7.38 mm
- net Net-(U3-LDOO): track 5.98 -> 7.01 mm
- net LRCLK1: track 18.3 -> 17.4 mm, vias 1 -> 0
- net BCLK1: track 18.1 -> 17.2 mm
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Other:
- board text added: "CTRL"
- board text removed: "I2C"
