File: PCBs/AURORA/DAC/1.0/DAC.kicad_sch (KiCad schematic)
At the start: 67 parts, among them J1 Conn_01x03_Pin, J10 Conn_01x02_Pin, J2 Conn_01x03_Pin, J3 Conn_01x03_Pin, J4 Conn_01x02_Pin, J5 Conn_01x03_Pin, J6 Conn_01x02_Pin, J7 Conn_01x04_Pin, J8 Conn_01x04_Pin, J9 Conn_01x04_Pin, U1 DA101C_C6931652, U2 AMS1117-3.3, U3 PCM5122PW, U4 PCM5122PW, U5 PCM5122PW

Commit message: Updates to amplifer
Parts:
- D1: value PURPLE -> RED; footprint Diode_SMD:D_0805_2012Metric -> LED_SMD:LED_0603_1608Metric
- D2: footprint Diode_SMD:D_0805_2012Metric -> LED_SMD:LED_0603_1608Metric
- R7: renamed from R6; value 300R -> 1.3K
- R8: renamed from R7; value 75R -> 150R
- renumbered C9 to C10, C10 to C11, C11 to C12, C12 to C13, C13 to C14, C14 to C15, C15 to C16, C16 to C17, C17 to C18, C18 to C19, C19 to C20, C20 to C21, C21 to C22, C22 to C23, C23 to C24, C24 to C25, C25 to C26, C26 to C27, C27 to C28, C28 to C29, C29 to C30, C30 to C31, C31 to C32, C32 to C33, C33 to C34, C34 to C35, C35 to C36, C36 to C37, C37 to C38, C38 to C5, C5 to C7, C7 to C8, C8 to C9, R2 to R1, R3 to R2, R4 to R3, R5 to R4, R8 to R5, R1 to R6
