File: PCBs/AURORA/DSP/STM32/0.2/DSP.kicad_pcb (KiCad board)
At the start: 4 copper layers, 85 x 55 mm, 86 parts, among them J1 Conn_01x04_Pin, J11 Conn_01x02_Pin, J13 Conn_01x04_Pin, J14 Conn_01x02_Pin, J15 Conn_01x02_Pin, J16 Conn_01x02_Pin, J17 Conn_01x02_Pin, J18 Conn_01x04_Pin, J19 Conn_01x05_Pin, J2 Conn_01x04_Pin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

Commit message: Moving files
Parts:
- removed J16: Conn_01x02_Pin, Connector_PinHeader_2.54mm:PinHeader_1x02_P2.54mm_Vertical
- added J8: Conn_01x03_Pin, Connector_PinHeader_2.54mm:PinHeader_1x03_P2.54mm_Vertical, F.Cu at (73.4, 82.0)
- added U6: ESP32-WROOM-32U, RF_Module:ESP32-WROOM-32U, F.Cu at (9.78, 9.88)
Connections:
- U5 pad 46: unconnected-(U5-PB10-Pad46) -> SPI_CLK
Routing:
- net SPI_CLK: track 0.00 -> 19.9 mm, vias 0 -> 2
