File: PCBs/AURORA/DSP/STM32/0.2/DSP.kicad_sch (KiCad schematic)
At the start: 86 parts, among them J1 Conn_01x04_Pin, J11 Conn_01x02_Pin, J13 Conn_01x04_Pin, J14 Conn_01x02_Pin, J15 Conn_01x02_Pin, J17 Conn_01x02_Pin, J18 Conn_01x04_Pin, J19 Conn_01x05_Pin, J2 Conn_01x04_Pin, J3 Conn_01x04_Pin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

Commit message: Moving files
Parts:
- added U6: ESP32-WROOM-32U, RF_Module:ESP32-WROOM-32U, symbol RF_Module:ESP32-WROOM-32U
Connections:
- new net: U6.1 (GND), U6.15 (GND), U6.38 (GND), U6.39 (GND)
