File: PCBs/AURORA/Microprocessor/1.0/uProcessor.kicad_pcb (KiCad board)
At the start: 2 copper layers, 85 x 55 mm, 66 parts, among them J1 Conn_01x02_Male, J10 Conn_01x02_Male, J11 Conn_01x02_Male, J12 Conn_01x02_Male, J13 Conn_01x03_Pin, J14 Conn_01x04_Pin, J15 Conn_01x04_Pin, J16 Conn_01x02_Male, J17 Conn_01x04_Pin, J2 Conn_01x05_Pin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

Commit message: Moving files
Parts:
- removed SW1: TS-1187A-B-A-B, easyeda2kicad:SW-SMD_4P-L5.1-W5.1-P3.70-LS6.5-TL_H1.5
- removed U2: ESP32-WROOM-32, PCM_Espressif:ESP32-WROOM-32E
- added J18: Conn_01x02_Male, Connector_JST:JST_PH_B2B-PH-K_1x02_P2.00mm_Vertical, F.Cu at (92.3, 97.9)
- added J19: Conn_01x02_Male, Connector_JST:JST_PH_B2B-PH-K_1x02_P2.00mm_Vertical, F.Cu at (160.1, 66.4)
- added R24: 150R, Resistor_SMD:R_0603_1608Metric_Pad0.98x0.95mm_HandSolder, F.Cu at (100.0, 90.5)
- added U4: ESP32-S3-WROOM-1, PCM_Espressif:ESP32-S3-WROOM-1, F.Cu at (131.9, 73.0)
- C1: value 10U -> 10N; footprint Capacitor_SMD:C_1206_3216Metric_Pad1.33x1.80mm_HandSolder -> Capacitor_SMD:C_0805_2012Metric_Pad1.18x1.45mm_HandSolder
- C2: value 10N -> 10U; footprint Capacitor_SMD:C_0805_2012Metric_Pad1.18x1.45mm_HandSolder -> Capacitor_SMD:C_1206_3216Metric_Pad1.33x1.80mm_HandSolder
- J14, J17: value Conn_01x04_Pin -> Conn_01x05_Pin; footprint Connector_JST:JST_PH_B4B-PH-K_1x04_P2.00mm_Vertical -> Connector_JST:JST_PH_B5B-PH-K_1x05_P2.00mm_Vertical
- moved R6 37.0 mm to (153.4, 108.2)
- moved R7 37.0 mm to (155.3, 108.2)
- moved D1 37.0 mm to (153.3, 104.8)
- moved D2 37.0 mm to (155.3, 104.8)
- moved Q2 8.82 mm to (133.8, 107.2)
- moved R21 8.82 mm to (136.2, 104.3)
- moved R22 8.82 mm to (129.5, 107.5)
- moved R23 8.82 mm to (137.3, 107.5)
- moved C11 6.00 mm to (145.0, 107.5)
- moved C12 6.00 mm to (147.1, 107.5)
- moved R10 5.54 mm to (145.8, 77.1)
- moved R13 5.54 mm to (145.8, 79.0)
- moved C4 5.05 mm to (155.2, 82.6)
- moved C6 5.05 mm to (155.2, 90.4)
- moved U3 5.05 mm to (153.4, 86.5)
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Routing:
- net GND: track 0.00 -> 384.3 mm, vias 0 -> 14
- net 3V3: track 0.00 -> 260.8 mm, vias 0 -> 5
- net 5V: track 0.00 -> 158.5 mm, vias 0 -> 2
- net ENABLE: track 0.00 -> 125.6 mm, vias 0 -> 1
- net SCL: track 0.00 -> 105.6 mm, vias 0 -> 2
- net SDA: track 0.00 -> 100.1 mm, vias 0 -> 3
- net SDA_5V: track 0.00 -> 90.9 mm, vias 0 -> 2
- net SCL_5V: track 0.00 -> 81.6 mm, vias 0 -> 1
- net BOOT: track 0.00 -> 55.5 mm, vias 0 -> 2
- net INPUT_CH2: track 0.00 -> 52.3 mm, vias 0 -> 1
- net INPUT_CH1: track 0.00 -> 52.0 mm, vias 0 -> 1
- net SD_CD: track 0.00 -> 50.0 mm, vias 0 -> 2
- net STANDBY_LED: track 0.00 -> 48.1 mm, vias 0 -> 2
- net SPI_CLK: track 0.00 -> 47.8 mm, vias 0 -> 2
- net SPI_CS: track 0.00 -> 46.6 mm, vias 0 -> 2
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- added copper zone on B.Cu, net GND
- added copper zone on F.Cu, net GND
- removed copper zone on B.Cu, net (none)
- removed copper zone on F.Cu, net (none)
Other:
- board text added: "RX/TX"
- board text added: "SBY_LED"
