File: PCBs/AURORA/Microprocessor/1.0/uProcessor.kicad_sch (KiCad schematic)
At the start: 66 parts, among them J1 Conn_01x02_Male, J10 Conn_01x02_Male, J11 Conn_01x02_Male, J12 Conn_01x02_Male, J13 Conn_01x03_Pin, J14 Conn_01x04_Pin, J15 Conn_01x04_Pin, J16 Conn_01x02_Male, J17 Conn_01x04_Pin, J2 Conn_01x05_Pin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

Commit message: Moving files
Parts:
- removed J14, J17: Conn_01x04_Pin, Connector_JST:JST_PH_B4B-PH-K_1x04_P2.00mm_Vertical, symbol Connector:Conn_01x04_Pin
- removed SW1: TS-1187A-B-A-B, easyeda2kicad:SW-SMD_4P-L5.1-W5.1-P3.70-LS6.5-TL_H1.5, symbol easyeda2kicad:TS-1187A-B-A-B
- removed U2: ESP32-WROOM-32, PCM_Espressif:ESP32-WROOM-32E, symbol RF_Module:ESP32-WROOM-32
- added J14, J17: Conn_01x05_Pin, Connector_JST:JST_PH_B5B-PH-K_1x05_P2.00mm_Vertical, symbol Connector:Conn_01x05_Pin
- added J18, J19: Conn_01x02_Male, Connector_JST:JST_PH_B2B-PH-K_1x02_P2.00mm_Vertical, symbol Connector:Conn_01x02_Male
- added R24: 150R, Resistor_SMD:R_0603_1608Metric_Pad0.98x0.95mm_HandSolder, symbol Device:R_Small
- added U4: ESP32-S3-WROOM-1, PCM_Espressif:ESP32-S3-WROOM-1, symbol PCM_Espressif:ESP32-S3-WROOM-1
- C1: value 10U -> 10N; footprint Capacitor_SMD:C_1206_3216Metric_Pad1.33x1.80mm_HandSolder -> Capacitor_SMD:C_0805_2012Metric_Pad1.18x1.45mm_HandSolder
- C2: value 10N -> 10U; footprint Capacitor_SMD:C_0805_2012Metric_Pad1.18x1.45mm_HandSolder -> Capacitor_SMD:C_1206_3216Metric_Pad1.33x1.80mm_HandSolder
Connections:
- net 3V3: now also J14.2 (Pin_2), J17.2 (Pin_2), U4.2 (3V3)
- net BACKLIGHT: now also U4.22 (GPIO14/TOUCH14/ADC2_CH3/FSPIWP/FSPIDQS/SUBSPIWP)
- net BOOT: now also U4.27 (GPIO0/BOOT)
- net ENABLE: now also U4.3 (EN)
- net GND: now also J14.1 (Pin_1), J17.1 (Pin_1), J18.1 (Pin_1), U4.1 (GND), U4.40 (GND), U4.41 (GND)
- net GPIO_INTA: now also U4.4 (GPIO4/TOUCH4/ADC1_CH3)
- net GPIO_INTB: now also U4.5 (GPIO5/TOUCH5/ADC1_CH4)
- net GPIO_RESET: now also U4.6 (GPIO6/TOUCH6/ADC1_CH5)
- net HARD_RESET: now also U4.7 (GPIO7/TOUCH7/ADC1_CH6)
- net INPUT_CH1: now also J17.3 (Pin_3), U4.23 (GPIO21)
- net INPUT_CH2: now also J17.4 (Pin_4), U4.24 (GPIO47/SPICLK_P/SUBSPICLK_P_DIFF)
- net IR_RECV: now also U4.8 (GPIO15/U0RTS/ADC2_CH4/XTAL_32K_P)
- net POWER_BUTTON: now also U4.10 (GPIO17/U1TXD/ADC2_CH6)
- net POWER_LED: now also U4.9 (GPIO16/U0CTS/ADC2_CH5/XTAL_32K_N)
- net RX: now also U4.36 (U0RXD/GPIO44/CLK_OUT2)
- net SCL: now also U4.33 (MTDO/GPIO40/CLK_OUT2)
- net SDA: now also U4.32 (MTCK/GPIO39/CLK_OUT3/SUBSPICS1)
- net SD_CD: now also U4.11 (GPIO18/U1RXD/ADC2_CH7/CLK_OUT3)
- net SPI_CLK: now also U4.18 (GPIO10/TOUCH10/ADC1_CH9/FSPICS0/FSPIIO4/SUBSPICS0)
- net SPI_CS: now also U4.17 (GPIO9/TOUCH9/ADC1_CH8/FSPIHD/SUBSPIHD)
- net SPI_MISO: now also U4.12 (GPIO8/TOUCH8/ADC1_CH7/SUBSPICS1)
- net SPI_MOSI: now also U4.15 (GPIO3/TOUCH3/ADC1_CH2)
- net TX: now also U4.37 (U0TXD/GPIO43/CLK_OUT1)
- net VOL_CH1: now also J14.3 (Pin_3), U4.19 (GPIO11/TOUCH11/ADC2_CH0/FSPID/FSPIIO5/SUBSPID)
- net VOL_CH2: now also J14.4 (Pin_4), U4.20 (GPIO12/TOUCH12/ADC2_CH1/FSPICLK/FSPIIO6/SUBSPICLK)
- net at R5.1: now also U4.34 (MTDI/GPIO41/CLK_OUT1)
- net at R4.1: now also U4.35 (MTMS/GPIO42)
- net at R3.1: now also U4.38 (GPIO2/TOUCH2/ADC1_CH1)
- net at R2.1: now also U4.39 (GPIO1/TOUCH1/ADC1_CH0)
- new net: J18.2 (Pin_2), R24.2
- new net DONTUSE3: U4.26 (GPIO45)
- new net DONTUSE4: U4.16 (GPIO46)
- new net INPUT_BUTTON: J17.5 (Pin_5), U4.25 (GPIO48/SPICLK_N/SUBSPICLK_N_DIFF)
- new net RX2: J19.2 (Pin_2), U4.30 (SPIDQS/GPIO37/FSPIQ/SUBSPIQ)
- new net STANDBY_LED: R24.1, U4.28 (SPIIO6/GPIO35/FSPID/SUBSPID)
- new net TX2: J19.1 (Pin_1), U4.29 (SPIIO7/GPIO36/FSPICLK/SUBSPICLK)
- new net USB_D+: U4.14 (GPIO20/U1CTS/ADC2_CH9/CLK_OUT1/USB_D+)
- new net USB_D-: U4.13 (GPIO19/U1RTS/ADC2_CH8/CLK_OUT2/USB_D-)
- new net VOL_BUTTON: J14.5 (Pin_5), U4.21 (GPIO13/TOUCH13/ADC2_CH2/FSPIQ/FSPIIO7/SUBSPIQ)
Other:
- moved on the sheet: C5, R21, R9, U1
