File: PCBs/AURORA/Extend/1.0/Extend.kicad_sch (KiCad schematic)
At the start: 27 parts, among them J1 Conn_01x05_Pin, J10 Conn_01x02_Male, J11 Conn_01x02_Male, J12 Conn_01x02_Male, J13 Conn_01x04_Pin, J2 Conn_01x05_Pin, J3 Conn_01x04_Pin, J5 Conn_01x02_Male, J6 Conn_01x02_Male, J7 Conn_01x02_Pin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

Commit message: Moving files
Parts:
- removed C2: 0.1u, Capacitor_SMD:C_0805_2012Metric_Pad1.18x1.45mm_HandSolder, symbol Device:C_Small
- removed J1: Conn_01x05_Pin, Connector_JST:JST_PH_B5B-PH-K_1x05_P2.00mm_Vertical, symbol Connector:Conn_01x05_Pin
- removed J10, J11, J12: Conn_01x02_Male, Connector_JST:JST_PH_B2B-PH-K_1x02_P2.00mm_Vertical, symbol Connector:Conn_01x02_Male
- removed R4: 320R, Resistor_SMD:R_0603_1608Metric_Pad0.98x0.95mm_HandSolder, symbol Device:R_Small
- removed U2: MCP23017_SS, Package_SO:SSOP-28_5.3x10.2mm_P0.65mm, symbol Interface_Expansion:MCP23017_SS
- added J1: Conn_01x06_Pin, Connector_JST:JST_PH_B6B-PH-K_1x06_P2.00mm_Vertical, symbol Connector:Conn_01x06_Pin
Connections:
- net INPUT_BUTTON is gone; now on net SPDIF_RESET: U1.8 (GPB7)
- net VOLUME_BUTTON is gone; now on net SPDIF_INT2: U1.7 (GPB6)
- net INTA: now also U1.20 (INTA); no longer U1.19 (INTB)
- net INTB: now also U1.19 (INTB)
- net SCL: now also J1.1 (Pin_1)
- net SDA: now also J1.2 (Pin_2)
- net SPDIF_INT1: now also U1.6 (GPB5)
- net DSP_EN1: now reaches U1.25 (GPA4)
- net DSP_EN1: now also J1.3 (Pin_3)
- net DSP_BOOT0 renamed DSP_EN3
- net DSP_EN3: now also J1.5 (Pin_5)
- net DSP_INT renamed DSP_BOOT
- net DSP_BOOT: now also J1.6 (Pin_6)
- net DSP_NRST renamed DSP_EN2
- net DSP_EN2: now also J1.4 (Pin_4)

Commit message: Replacing PeakingEQ
Parts:
- added J10, J4: Conn_01x02_Male, Connector_JST:JST_PH_B2B-PH-K_1x02_P2.00mm_Vertical, symbol Connector:Conn_01x02_Male
- added R4: 4.7K, Resistor_SMD:R_0603_1608Metric_Pad0.98x0.95mm_HandSolder, symbol Device:R_Small
Connections:
- net GND: now also J10.1 (Pin_1), J4.1 (Pin_1), R4.1
- net MONOBLOCK_ENABLE: now reaches U1.23 (GPA2)
- net MONOBLOCK_ENABLE: now also J10.2 (Pin_2), J4.2 (Pin_2), R4.2
